File: RAM128.kicad_sch (KiCad schematic)
At the start: 50 parts, among them J1 AppleIIBus, SW1 DMA/ROM, U1 621024, U10 74AHCT32PW, U11 74LVC1G126GW, U12 74AHCT1G04GW, U13 74AHCT1G04GW, U14 74AHCT1G04GW, U15 74AHCT1G04GW, U16 74AHCT1G04GW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

Commit message: As submitted to JLC
Parts:
- U1: footprint stdpads:SOP-32_P1.27mm -> stdpads:SOP-32_450mil
Connections:
- no-connect marks 11 -> 12
Changed lines of the file:
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@@
   )
   (no_connect (at 254 36.83))
+  (no_connect (at 87.63 90.17))
   (no_connect (at 248.92 80.01))
   (no_connect (at 254 34.29))
@@
     (property "Reference" "U1" (id 0) (at 97.79 60.96 0))
     (property "Value" "621024" (id 1) (at 97.79 85.09 90))
-    (property "Footprint" "stdpads:SOP-32_P1.27mm" (id 2) (at 97.79 85.09 0)
+    (property "Footprint" "stdpads:SOP-32_450mil" (id 2) (at 97.79 85.09 0)
       (effects (font (size 1.27 1.27)) hide)
     )
@@
     )
     (path "/00000000-0000-0000-0000-000061c2b655"
-      (reference "U1") (unit 1) (value "621024") (footprint "stdpads:SOP-32_P1.27mm")
+      (reference "U1") (unit 1) (value "621024") (footprint "stdpads:SOP-32_450mil")
     )
     (path "/00000000-0000-0000-0000-00005f96867c"

Commit message: Draft 4208C
Parts:
- removed SW1: DMA/ROM, stdpads:SW_DIP_SPSTx02_Slide_DSHP02TS_P1.27mm, symbol Switch:SW_DIP_x02
- added R6: 10k, stdpads:R_0805, symbol Device:R_Small
- added SW1: DMA/ROM/SIZE, stdpads:SW_DIP_SPSTx03_Slide_DSHP03TS_P1.27mm, symbol Switch:SW_DIP_x03
- U11: value 74LVC1G126GW -> 74AHCT1G126GW
Connections:
- net +5V: now also R6.1
- net DMAin: now also SW1.6
- net RCS: now also SW1.5
- net ~{A2}: now also SW1.4; no longer U7.1
- net at R2.1, U7.9: now also SW1.2
- net at R4.2, U6.13: now also SW1.1
- new net ~{A2}g: R6.2, SW1.3, U7.1
Other:
- title: RAM128 (GW4208B) -> RAM128 (GW4208C)
- moved on the sheet: R3, U7A
