File: RAM128.kicad_sch (KiCad schematic)
At the start: 50 parts, among them J1 AppleIIBus, SW1 DMA/ROM, U1 621024, U10 74AHCT32PW, U11 74LVC1G126GW, U12 74AHCT1G04GW, U13 74AHCT1G04GW, U14 74AHCT1G04GW, U15 74AHCT1G04GW, U16 74AHCT1G04GW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

Commit message: 1.1?
Parts:
- H1, H2, H3, H4, H5: symbol Mechanical:MountingHole_Pad -> Mechanical:MountingHole
Connections:
- net GND: no longer H1.1, H2.1, H3.1, H4.1, H5.1

Commit message: 1.2?
Parts:
- added C17: 2u2, stdpads:C_0603, symbol Device:C_Small
Connections:
- net +5V: now also C17.1
- net A13: no longer U7.13
- net D0: now also U2.9 (A7); no longer U2.18 (B0)
- net D1: now also U2.8 (A6); no longer U2.17 (B1)
- net D2: now also U2.7 (A5); no longer U2.16 (B2)
- net D3: now also U2.6 (A4); no longer U2.15 (B3)
- net D4: now also U2.5 (A3); no longer U2.14 (B4)
- net D5: now also U2.4 (A2); no longer U2.13 (B5)
- net D6: now also U2.3 (A1); no longer U2.12 (B6)
- net D7: now also U2.2 (A0); no longer U2.11 (B7)
- net GND: now also C17.2
- net Q3: now also U2.19 (~{OE})
- net RD0: now also U2.15 (B3); no longer U2.6 (A4)
- net RD1: now also U2.17 (B1); no longer U2.8 (A6)
- net RD2: now also U2.12 (B6); no longer U2.3 (A1)
- net RD3: now also U2.11 (B7); no longer U2.2 (A0)
- net RD4: now also U2.13 (B5); no longer U2.4 (A2)
- net RD5: now also U2.18 (B0); no longer U2.9 (A7)
- net RD6: now also U2.16 (B2); no longer U2.7 (A5)
- net RD7: now also U2.14 (B4); no longer U2.5 (A3)
- net R~{CS}: now also U7.13; no longer U2.19 (~{OE})
- net R~{W}: no longer U2.1 (AtoB), U7.12
- net ~{R}W: now also U7.12
- net DDIR: now reaches U7.11
- net DDIR: now also U2.1 (AtoB)
- net at U9.11: no longer U10.9
- no-connect marks 12 -> 11
Other:
- moved on the sheet: C16, R1, R3, R4, R5, SW1, U10A, U10B, U10C, U10D, U11, U12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

Commit message: 1.2?
Parts:
- removed C17: 2u2, stdpads:C_0603, symbol Device:C_Small
Connections:
- net at U9.11: now also U10.9
Other:
- moved on the sheet: C16
Changed lines of the file:
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@@
   (junction (at 120.65 189.23) (diameter 0) (color 0 0 0 0)
   )
+  (junction (at 110.49 168.91) (diameter 0) (color 0 0 0 0)
+  )
   (junction (at 140.97 184.15) (diameter 0) (color 0 0 0 0)
   )
@@
   (junction (at 220.98 102.87) (diameter 0) (color 0 0 0 0)
   )
-  (junction (at 110.49 173.99) (diameter 0) (color 0 0 0 0)
-  )
   (junction (at 104.14 139.7) (diameter 0) (color 0 0 0 0)
   )
@@
   (junction (at 140.97 179.07) (diameter 0) (color 0 0 0 0)
   )
-  (junction (at 110.49 168.91) (diameter 0) (color 0 0 0 0)
-  )
   (junction (at 231.14 41.91) (diameter 0) (color 0 0 0 0)
   )
-  (junction (at 100.33 168.91) (diameter 0) (color 0 0 0 0)
-  )
   (junction (at 45.72 172.72) (diameter 0) (color 0 0 0 0)
   )
@@
     (stroke (width 0) (type default))
   )
-  (wire (pts (xy 100.33 168.91) (xy 110.49 168.91))
-    (stroke (width 0) (type default))
-  )
   (wire (pts (xy 261.62 31.75) (xy 256.54 31.75))
     (stroke (width 0) (type default))
@@
     (stroke (width 0) (type default))
   )
-  (wire (pts (xy 165.1 99.06) (xy 165.1 101.6))
+  (wire (pts (xy 165.1 87.63) (xy 165.1 90.17))
     (stroke (width 0) (type default))
   )
@@
     (stroke (width 0) (type default))
   )
-  (wire (pts (xy 100.33 173.99) (xy 110.49 173.99))
-    (stroke (width 0) (type default))
-  )
   (bus (pts (xy 115.57 80.01) (xy 115.57 82.55))
     (stroke (width 0) (type default))
@@
     (stroke (width 0) (type default))
   )
-  (wire (pts (xy 134.62 134.62) (xy 134.62 134.62))
-    (stroke (width 0) (type default))
-  )
   (wire (pts (xy 215.9 77.47) (xy 215.9 80.01))
     (stroke (width 0) (type default))
@@
     )
   )
-  (symbol (lib_id "Device:C_Small") (at 90.17 171.45 0) (unit 1)
+  (symbol (lib_id "Device:C_Small") (at 100.33 171.45 0) (unit 1)
     (in_bom yes) (on_board yes) (dnp no)
-    (property "Reference" "C16" (at 91.44 170.18 0)
+    (property "Reference" "C16" (at 101.6 170.18 0)
       (effects (font (size 1.27 1.27)) (justify left))
     )
-    (property "Value" "10u" (at 91.44 172.72 0)
+    (property "Value" "10u" (at 101.6 172.72 0)
       (effects (font (size 1.27 1.27)) (justify left))
     )
-    (property "Footprint" "stdpads:C_0805" (at 90.17 171.45 0)
+    (property "Footprint" "stdpads:C_0805" (at 100.33 171.45 0)
       (effects (font (size 1.27 1.27)) hide)
     )
-    (property "Datasheet" "~" (at 90.17 171.45 0)
+    (property "Datasheet" "~" (at 100.33 171.45 0)
       (effects (font (size 1.27 1.27)) hide)
     )
-    (property "LCSC Part" "C15850" (at 90.17 171.45 0)
+    (property "LCSC Part" "C15850" (at 100.33 171.45 0)
       (effects (font (size 1.27 1.27)) hide)
     )
@@
     )
   )
-  (symbol (lib_id "power:+12V") (at 90.17 168.91 0) (mirror y) (unit 1)
+  (symbol (lib_id "power:+12V") (at 100.33 168.91 0) (mirror y) (unit 1)
     (in_bom yes) (on_board yes) (dnp no)
-    (property "Reference" "#PWR0128" (at 90.17 172.72 0)
+    (property "Reference" "#PWR0128" (at 100.33 172.72 0)
       (effects (font (size 1.27 1.27)) hide)
     )
-    (property "Value" "+12V" (at 90.17 165.1 0)
+    (property "Value" "+12V" (at 100.33 165.1 0)
       (effects (font (size 1.27 1.27)))
     )
-    (property "Footprint" "" (at 90.17 168.91 0)
+    (property "Footprint" "" (at 100.33 168.91 0)
       (effects (font (size 1.27 1.27)) hide)
     )
-    (property "Datasheet" "" (at 90.17 168.91 0)
+    (property "Datasheet" "" (at 100.33 168.91 0)
       (effects (font (size 1.27 1.27)) hide)
     )
@@
     )
   )
-  (symbol (lib_id "power:GND") (at 90.17 173.99 0) (unit 1)
+  (symbol (lib_id "power:GND") (at 100.33 173.99 0) (unit 1)
     (in_bom yes) (on_board yes) (dnp no)
-    (property "Reference" "#PWR0146" (at 90.17 180.34 0)
+    (property "Reference" "#PWR0146" (at 100.33 180.34 0)
       (effects (font (size 1.27 1.27)) hide)
     )
-    (property "Value" "GND" (at 90.17 177.8 0)
+    (property "Value" "GND" (at 100.33 177.8 0)
       (effects (font (size 1.27 1.27)))
     )
-    (property "Footprint" "" (at 90.17 173.99 0)
+    (property "Footprint" "" (at 100.33 173.99 0)
       (effects (font (size 1.27 1.27)) hide)
     )
-    (property "Datasheet" "" (at 90.17 173.99 0)
+    (property "Datasheet" "" (at 100.33 173.99 0)
       (effects (font (size 1.27 1.27)) hide)
     )
@@
     )
   )
-  (symbol (lib_id "power:+5V") (at 100.33 168.91 0) (unit 1)
+  (symbol (lib_id "power:+5V") (at 110.49 168.91 0) (unit 1)
     (in_bom yes) (on_board yes) (dnp no)
-    (property "Reference" "#PWR03" (at 100.33 172.72 0)
+    (property "Reference" "#PWR03" (at 110.49 172.72 0)
       (effects (font (size 1.27 1.27)) hide)
     )
-    (property "Value" "+5V" (at 100.33 165.1 0)
+    (property "Value" "+5V" (at 110.49 165.1 0)
       (effects (font (size 1.27 1.27)))
     )
-    (property "Footprint" "" (at 100.33 168.91 0)
+    (property "Footprint" "" (at 110.49 168.91 0)
       (effects (font (size 1.27 1.27)) hide)
     )
-    (property "Datasheet" "" (at 100.33 168.91 0)
+    (property "Datasheet" "" (at 110.49 168.91 0)
       (effects (font (size 1.27 1.27)) hide)
     )
@@
         )
       )
-    )
-  )
-  (symbol (lib_id "Device:C_Small") (at 100.33 171.45 0) (unit 1)
-    (in_bom yes) (on_board yes) (dnp no)
-    (property "Reference" "C17" (at 101.6 170.18 0)
-      (effects (font (size 1.27 1.27)) (justify left))
-    )
-    (property "Value" "2u2" (at 101.6 172.72 0)
-      (effects (font (size 1.27 1.27)) (justify left))
-    )
-    (property "Footprint" "stdpads:C_0603" (at 100.33 171.45 0)
-      (effects (font (size 1.27 1.27)) hide)
-    )
-    (property "Datasheet" "~" (at 100.33 171.45 0)
-      (effects (font (size 1.27 1.27)) hide)
-    )
-    (property "LCSC Part" "C23630" (at 100.33 171.45 0)
-      (effects (font (size 1.27 1.27)) hide)
-    )
-    (pin "1")
-    (pin "2")
-    (instances
-      (project "RAM128"
-        (path "/b0906e10-2fbc-4309-a8b4-6fc4cd1a5490"
-          (reference "C17") (unit 1)
-        )
-      )
