File: RAM128.kicad_sch (KiCad schematic)
At the start: 50 parts, among them J1 AppleIIBus, SW1 DMA/ROM, U1 621024, U10 74AHCT32PW, U11 74LVC1G126GW, U12 74AHCT1G04GW, U13 74AHCT1G04GW, U14 74AHCT1G04GW, U15 74AHCT1G04GW, U16 74AHCT1G04GW, U17 74AHCT1G04GW, U19 74AHCT1G04GW, U2 74HCT245PW, U20 74AHCT1G04GW, U3 74HCT273PW, U4 74HCT273PW, U6 74AHCT08PW, U7 74AHCT32PW, U8 74AHCT08PW, U9 74AHCT08PW

Commit message: 1.2 RC2
Parts:
- added C17, C18: 2u2, stdpads:C_0603, symbol Device:C_Small
- added R6: DNP, stdpads:R_0805, symbol Device:R_Small
- added U18, U5: 74AHCT1G32GW, stdpads:SOT-353, symbol GW_Logic:741G32GW
- R5: value 33 -> 0; LCSC Part C17634 -> C17477
- U11: value 74LVC1G126GW -> 74AHCT1G126GW; LCSC Part C88039 -> C150723
Connections:
- net +5V: now also C17.1, C18.1, U18.5 (Vcc), U5.5 (Vcc)
- net GND: now also C17.2, C18.2, U18.3 (GND), U5.3 (GND); no longer U1.24 (~{OE})
- net PHI1: now also U5.1 (A)
- net Q3: now also U5.2 (B); no longer U2.19 (~{OE})
- net R~{W}: now also R6.1, U18.1 (A); no longer U1.29 (~{WE})
- net ~{R}W: now also U1.24 (~{OE})
- new net D~{OE}: U18.2 (B), U2.19 (~{OE}), U5.4 (Y)
- new net R~{WE}: R6.2, U1.29 (~{WE}), U18.4 (Y)
Other:
- moved on the sheet: C1, C16

Commit message: 1.2 RC4
Parts:
- R1: value 3k3 -> 22k; LCSC Part C26010 -> C17560
- R3: value 10k -> 22k; LCSC Part C17414 -> C17560
Changed lines of the file:
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@@
   (junction (at 120.65 179.07) (diameter 0) (color 0 0 0 0)
   )
-  (junction (at 226.06 107.95) (diameter 0) (color 0 0 0 0)
-  )
   (junction (at 110.49 189.23) (diameter 0) (color 0 0 0 0)
   )
@@
   (junction (at 224.79 82.55) (diameter 0) (color 0 0 0 0)
   )
+  (junction (at 104.14 134.62) (diameter 0) (color 0 0 0 0)
+  )
   (junction (at 33.02 172.72) (diameter 0) (color 0 0 0 0)
   )
-  (junction (at 220.98 102.87) (diameter 0) (color 0 0 0 0)
+  (junction (at 226.06 107.95) (diameter 0) (color 0 0 0 0)
   )
   (junction (at 104.14 139.7) (diameter 0) (color 0 0 0 0)
@@
   (junction (at 45.72 172.72) (diameter 0) (color 0 0 0 0)
   )
+  (junction (at 220.98 102.87) (diameter 0) (color 0 0 0 0)
+  )
   (junction (at 33.02 198.12) (diameter 0) (color 0 0 0 0)
   )
@@
   (junction (at 140.97 189.23) (diameter 0) (color 0 0 0 0)
   )
-  (junction (at 104.14 134.62) (diameter 0) (color 0 0 0 0)
-  )
   (junction (at 224.79 85.09) (diameter 0) (color 0 0 0 0)
   )
@@
     (stroke (width 0) (type default))
   )
-  (wire (pts (xy 220.98 102.87) (xy 226.06 102.87))
-    (stroke (width 0) (type default))
-  )
   (wire (pts (xy 231.14 36.83) (xy 231.14 39.37))
     (stroke (width 0) (type default))
@@
     (stroke (width 0) (type default))
   )
+  (wire (pts (xy 220.98 102.87) (xy 226.06 102.87))
+    (stroke (width 0) (type default))
+  )
   (wire (pts (xy 20.32 172.72) (xy 33.02 172.72))
     (stroke (width 0) (type default))
@@
     )
   )
-  (symbol (lib_id "Device:R_Small") (at 226.06 105.41 0) (unit 1)
-    (in_bom yes) (on_board yes) (dnp no)
-    (property "Reference" "R1" (at 227.5586 104.2416 0)
-      (effects (font (size 1.27 1.27)) (justify left))
-    )
-    (property "Value" "3k3" (at 227.5586 106.553 0)
-      (effects (font (size 1.27 1.27)) (justify left))
-    )
-    (property "Footprint" "stdpads:R_0805" (at 226.06 105.41 0)
-      (effects (font (size 1.27 1.27)) hide)
-    )
-    (property "Datasheet" "~" (at 226.06 105.41 0)
-      (effects (font (size 1.27 1.27)) hide)
-    )
-    (property "LCSC Part" "C26010" (at 226.06 105.41 0)
-      (effects (font (size 1.27 1.27)) hide)
-    )
-    (pin "1")
-    (pin "2")
-    (instances
-      (project "RAM128"
-        (path "/b0906e10-2fbc-4309-a8b4-6fc4cd1a5490"
-          (reference "R1") (unit 1)
-        )
-      )
-    )
-  )
   (symbol (lib_id "Device:C_Small") (at 80.01 171.45 0) (unit 1)
     (in_bom yes) (on_board yes) (dnp no)
@@
     )
   )
-  (symbol (lib_id "Device:R_Small") (at 104.14 137.16 0) (unit 1)
-    (in_bom yes) (on_board yes) (dnp no)
-    (property "Reference" "R3" (at 105.6386 135.9916 0)
-      (effects (font (size 1.27 1.27)) (justify left))
-    )
-    (property "Value" "10k" (at 105.6386 138.303 0)
-      (effects (font (size 1.27 1.27)) (justify left))
-    )
-    (property "Footprint" "stdpads:R_0805" (at 104.14 137.16 0)
-      (effects (font (size 1.27 1.27)) hide)
-    )
-    (property "Datasheet" "~" (at 104.14 137.16 0)
-      (effects (font (size 1.27 1.27)) hide)
-    )
-    (property "LCSC Part" "C17414" (at 104.14 137.16 0)
-      (effects (font (size 1.27 1.27)) hide)
-    )
-    (pin "1")
-    (pin "2")
-    (instances
-      (project "RAM128"
-        (path "/b0906e10-2fbc-4309-a8b4-6fc4cd1a5490"
-          (reference "R3") (unit 1)
-        )
-      )
-    )
-  )
   (symbol (lib_id "power:+5V") (at 104.14 134.62 0) (unit 1)
     (in_bom yes) (on_board yes) (dnp no)
@@
     )
   )
+  (symbol (lib_id "Device:R_Small") (at 104.14 137.16 0) (unit 1)
+    (in_bom yes) (on_board yes) (dnp no)
+    (property "Reference" "R3" (at 105.6386 135.9916 0)
+      (effects (font (size 1.27 1.27)) (justify left))
+    )
+    (property "Value" "22k" (at 105.6386 138.303 0)
+      (effects (font (size 1.27 1.27)) (justify left))
+    )
+    (property "Footprint" "stdpads:R_0805" (at 104.14 137.16 0)
+      (effects (font (size 1.27 1.27)) hide)
+    )
+    (property "Datasheet" "~" (at 104.14 137.16 0)
+      (effects (font (size 1.27 1.27)) hide)
+    )
+    (property "LCSC Part" "C17560" (at 104.14 137.16 0)
+      (effects (font (size 1.27 1.27)) hide)
+    )
+    (pin "1")
+    (pin "2")
+    (instances
+      (project "RAM128"
+        (path "/b0906e10-2fbc-4309-a8b4-6fc4cd1a5490"
+          (reference "R3") (unit 1)
+        )
+      )
+    )
+  )
   (symbol (lib_id "power:GND") (at 207.01 160.02 0) (unit 1)
     (in_bom yes) (on_board yes) (dnp no)
@@
         )
       )
+    )
+  )
+  (symbol (lib_id "Device:R_Small") (at 226.06 105.41 0) (unit 1)
+    (in_bom yes) (on_board yes) (dnp no)
+    (property "Reference" "R1" (at 227.5586 104.2416 0)
+      (effects (font (size 1.27 1.27)) (justify left))
+    )
+    (property "Value" "22k" (at 227.5586 106.553 0)
+      (effects (font (size 1.27 1.27)) (justify left))
+    )
+    (property "Footprint" "stdpads:R_0805" (at 226.06 105.41 0)
+      (effects (font (size 1.27 1.27)) hide)
+    )
+    (property "Datasheet" "~" (at 226.06 105.41 0)
+      (effects (font (size 1.27 1.27)) hide)
+    )
+    (property "LCSC Part" "C17560" (at 226.06 105.41 0)
+      (effects (font (size 1.27 1.27)) hide)
+    )
+    (pin "1")
+    (pin "2")
+    (instances
+      (project "RAM128"
+        (path "/b0906e10-2fbc-4309-a8b4-6fc4cd1a5490"
+          (reference "R1") (unit 1)
+        )
+      )

Commit message: Update BOM, no board changes
Parts:
- U18, U5: LCSC Part (none) -> C554582
Changed lines of the file:
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@@
       (effects (font (size 1.524 1.524)) hide)
+    )
+    (property "LCSC Part" "C554582" (at 247.65 160.02 0)
+      (effects (font (size 1.27 1.27)) hide)
     )
     (pin "1")
@@
       (effects (font (size 1.524 1.524)) hide)
     )
+    (property "LCSC Part" "C554582" (at 217.17 157.48 0)
+      (effects (font (size 1.27 1.27)) hide)
+    )
     (pin "1")

Commit message: idk
Parts:
- removed SW1: DMA/ROM, stdpads:SW_DIP_SPSTx02_Slide_DSHP02TS_P1.27mm, symbol Switch:SW_DIP_x02
- added C20: 2u2, stdpads:C_0603, symbol Device:C_Small
- added D1, D2, D3, D4, D5, D6: Amber, stdpads:LED_0805, symbol Device:LED_Small_ALT
- added R10, R7, R8, R9: 22k, stdpads:R_0805, symbol Device:R_Small
- added R11, R12, R13, R14, R15, R16: 470, stdpads:R_0805, symbol Device:R_Small
- added SW1: CFG, stdpads:SW_DIP_SPSTx05_Slide_DSHP05TS_P1.27mm, symbol Switch:SW_DIP_x05
- added U21, U22, U23, U25: 74AHCT1G04GW, stdpads:SOT-353, symbol GW_Logic:741G04GW
- added U24: 74AHCT1G32GW, stdpads:SOT-353, symbol GW_Logic:741G32GW
- added U26, U27, U28, U29, U30, U31: 74AHCT1G08GW, stdpads:SOT-353, symbol GW_Logic:741G08GW
- H1, H2, H3, H4, H5: value (none) -> ~
Connections:
- net +5V: now also R10.1, R9.1, U21.5 (Vcc), U22.5 (Vcc), U23.5 (Vcc), U24.5 (Vcc), U25.5 (Vcc), U26.5 (Vcc), U27.5 (Vcc), U28.5 (Vcc), U29.5 (Vcc), U30.5 (Vcc), U31.5 (Vcc)
- net A2: no longer U7.4
- net DMAin: now also SW1.1
- net ENRD: now also U29.1 (A)
- net ENWR: now also U30.1 (A)
- net GND: now also C20.2, D1.1 (K), D2.1 (K), D3.1 (K), D4.1 (K), D5.1 (K), D6.1 (K), R7.2, R8.2, U21.3 (GND), U22.3 (GND), U23.3 (GND), U24.3 (GND), U25.3 (GND), U26.3 (GND), U27.3 (GND), U28.3 (GND), U29.3 (GND), U30.3 (GND), U31.3 (GND)
- net RA14: now also U28.1 (A)
- net RA15: now also U27.1 (A)
- net RA16: now also U26.1 (A)
- net RCS: now also SW1.2, U31.1 (A)
- net ~{A2}: now also SW1.3
- net ~{RES}: now also U23.2 (A); no longer U3.1 (~{Mr}), U4.1 (~{Mr})
- net RCSsw: now reaches R2.1, U7.9
- net RCSsw: now also SW1.9
- net DMAinsw: now reaches R4.2, U6.13
- net DMAinsw: now also SW1.10
- new net: R11.2, U26.4 (Y)
- new net: R15.2, U30.4 (Y)
- new net: R13.2, U28.4 (Y)
- new net: R16.2, U31.4 (Y)
- new net: R12.2, U27.4 (Y)
- new net: R9.2, SW1.6
- new net: R14.2, U29.4 (Y)
- new net BA2: U21.4 (Y), U7.4
- new net LEDEN: R7.1, SW1.5, U26.2 (B), U27.2 (B), U28.2 (B), U29.2 (B), U30.2 (B), U31.2 (B)
- new net LED_ACT: D6.2 (A), R16.1
- new net LED_ENRD: D4.2 (A), R14.1
- new net LED_ENWR: D5.2 (A), R15.1
- new net LED_RA14: D3.2 (A), R13.1
- new net LED_RA15: D2.2 (A), R12.1
- new net LED_RA16: D1.2 (A), R11.1
- new net PUP: U22.4 (Y), U24.1 (A)
- new net RES: SW1.4, U23.4 (Y)
- new net RESsw: R8.1, SW1.7, U24.2 (B)
- new net RRST: U24.4 (Y), U25.2 (A)
- new net ~{A2}sw: SW1.8, U21.2 (A)
- new net ~{PUP}: C20.1, R10.2, U22.2 (A)
- new net ~{RRST}: U25.4 (Y), U3.1 (~{Mr}), U4.1 (~{Mr})
- no-connect marks 11 -> 14
Other:
- moved on the sheet: H1, H2, H3, H4, H5, R4

Commit message: consolidate logic
Parts:
- removed D1, D2, D3, D4, D5, D6: Amber, stdpads:LED_0805, symbol Device:LED_Small_ALT
- removed J1: AppleIIBus, stdpads:AppleIIBus_Edge, symbol Connector_Generic:Conn_02x25_Counter_Clockwise
- removed R1: 22k, stdpads:R_0805, symbol Device:R_Small
- removed R11, R12, R13, R14, R15, R16: 470, stdpads:R_0805, symbol Device:R_Small
- removed R5: 0, stdpads:R_0805, symbol Device:R_Small
- removed R6: DNP, stdpads:R_0805, symbol Device:R_Small
- removed U1: 621024, stdpads:SOP-32_450mil, symbol GW_RAM:SRAM-128Kx8-SOP-32
- removed U11: 74AHCT1G126GW, stdpads:SOT-353, symbol GW_Logic:741G126GW
- removed U18, U24, U5: 74AHCT1G32GW, stdpads:SOT-353, symbol GW_Logic:741G32GW
- removed U19, U21, U25: 74AHCT1G04GW, stdpads:SOT-353, symbol GW_Logic:741G04GW
- removed U2: 74HCT245PW, stdpads:TSSOP-20_4.4x6.5mm_P0.65mm, symbol GW_Logic:74245
- removed U26, U27, U28, U29, U30, U31: 74AHCT1G08GW, stdpads:SOT-353, symbol GW_Logic:741G08GW
- removed U3, U4: 74HCT273PW, stdpads:TSSOP-20_4.4x6.5mm_P0.65mm, symbol 74xx:74LS273
- added U19: 74AHCT32PW, stdpads:TSSOP-14_4.4x5mm_P0.65mm, symbol 74xx:74LS32
- added U21: 74AHCT08PW, stdpads:TSSOP-14_4.4x5mm_P0.65mm, symbol 74xx:74LS02
- added U27: 74AHCT08PW, stdpads:TSSOP-14_4.4x5mm_P0.65mm, symbol 74xx:74LS08
Connections:
- net +5V: now also R2.1
- net A2: now also U7.10
- net BA2: now also SW1.3, U7.8
- net DMAin: now also U27.2
- net DMAout: now also U27.3; no longer U20.4 (Y)
- net D~{OE}: now also U19.11, U19.9
- net GND: now also U7.9; no longer R2.2
- net PHI1: now also U19.13
- net Q3: now also U19.12
- net RCS: no longer SW1.2
- net RESsw: now also U19.2
- net RRST: now also U20.2 (A), U19.3
- net R~{CS}: now also SW1.2
- net R~{WE}: now also U19.8
- net R~{W}: now also U19.10
- net ~{A2}: no longer SW1.3
- net ~{RRST}: now also U20.4 (Y)
- net PUP renamed POR
- net POR: now also U19.1
- removed net RCSsw: R2.1, SW1.9, U7.9
- net ~{A2}sw renamed BA2sw
- removed net ~{DMAout}: U20.2 (A), U7.8
- net ~{PUP} renamed ~{POR}
- new net R~{CS}sw: R2.2, SW1.9, U27.1
- no-connect marks 14 -> 2
Other:
- added sheet Buf (Buf.kicad_sch)
- added sheet Bus (Bus.kicad_sch)
- added sheet Control (Control.kicad_sch)
- added sheet LEDs (LEDs.kicad_sch)
- added sheet RAM (RAM.kicad_sch)
- added sheet Registers (Registers.kicad_sch)

Commit message: schematic and placement done?
Parts:
- removed C1, C16: 10u, stdpads:C_0805, symbol Device:C_Small
- removed C10, C11, C12, C13, C14, C15, C17, C18, C2, C20, C3, C4, C5, C6, C7, C8, C9: 2u2, stdpads:C_0603, symbol Device:C_Small
- removed R10, R2, R3, R4, R7, R8, R9: 22k, stdpads:R_0805, symbol Device:R_Small
- removed SW1: CFG, stdpads:SW_DIP_SPSTx05_Slide_DSHP05TS_P1.27mm, symbol Switch:SW_DIP_x05
- removed U10, U19, U7: 74AHCT32PW, stdpads:TSSOP-14_4.4x5mm_P0.65mm, symbol 74xx:74LS32
- removed U12, U13, U14, U15, U16, U17, U20, U22, U23: 74AHCT1G04GW, stdpads:SOT-353, symbol GW_Logic:741G04GW
- removed U21: 74AHCT08PW, stdpads:TSSOP-14_4.4x5mm_P0.65mm, symbol 74xx:74LS02
- removed U27, U6, U8, U9: 74AHCT08PW, stdpads:TSSOP-14_4.4x5mm_P0.65mm, symbol 74xx:74LS08
Connections:
- no-connect marks 2 -> 0
Other:
- added sheet Config (Config.kicad_sch)
- sheet Buf ports: added DDIR, D[7..0], D~{OE}, INH~{OE}, RD[7..0], ~{INH}; removed none
- sheet Bus ports: added A[15..0], DMAin, DMAout, D[7..0], PHI0, PHI1, Q3, R~{W}, ~{DEVSEL}, ~{INH}, ~{RESET}; removed none
- sheet Control ports: added A2clk, A2sw, A[15..0], BankAB, DDIR, DMAin, DMAinsw, DMAout, DMAoutEN, D~{OE}, ENRD, ENWR, ENWR1, ENWR1A0, INH~{OE}, PHI0, PHI1, Q3, RA12, RCS, RES, RESsw, R~{RST}, R~{WE}, R~{W}, ~{A0XOR1}, ~{A2}clk, ~{DEVSEL}, ~{RESET}, ~{R}W; removed none
- sheet LEDs ports: added ENRD, ENWR, LEDEN, RA14, RA15, RA16, RCS; removed none
- sheet RAM ports: added A[15..0], RA12, RA14, RA15, RA16, RCS, RD[7..0], R~{WE}, ~{R}W; removed none
- sheet Registers ports: added A2clk, A[15..0], BankAB, ENRD, ENWR, ENWR1, ENWR1A0, RA14, RA15, RA16, ~{A0XOR1}, ~{A2}clk, ~{RRST}; removed none
