File: RAM128.kicad_pcb (KiCad board)
At the start: 4 copper layers, 74.2 x 42.7 mm, 52 parts, among them J1 AppleIIBus, SW1 DMA/ROM, U1 621024, U10 74AHCT32PW, U11 74LVC1G126GW, U12 74AHCT1G04GW, U13 74AHCT1G04GW, U14 74AHCT1G04GW, U15 74AHCT1G04GW, U16 74AHCT1G04GW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

Commit message: 1.1?
Parts:
- moved G*** 0.12 mm to (125.6, 100.8)
- moved G*** 0.06 mm to (108.0, 100.9)
- turned U11 to 180 degrees
- turned U12 to 0 degrees
- turned U13 to 0 degrees
- turned U14 to 0 degrees
- turned U15 to 0 degrees
- turned U16 to 0 degrees
- turned U17 to 0 degrees
- turned U19 to 0 degrees
- turned U20 to 0 degrees
Other:
- board text added: "B11"
- board text added: "ZK, GF"

Commit message: 1.2?
Parts:
- moved C7 10.2 mm to (78.6, 118.0), turned to -90 degrees
- moved R2 1.20 mm to (101.3, 115.5)
- turned U2 to 0 degrees
Connections:
- U10 pad 9: Net-(U10-Pad9) -> unconnected-(U10-Pad9)
- U2 pad 1: /R~{W} -> /DDIR
- U2 pad 11: /D7 -> /RD3
- U2 pad 12: /D6 -> /RD2
- U2 pad 13: /D5 -> /RD4
- U2 pad 14: /D4 -> /RD7
- U2 pad 15: /D3 -> /RD0
- U2 pad 16: /D2 -> /RD6
- U2 pad 17: /D1 -> /RD1
- U2 pad 18: /D0 -> /RD5
- U2 pad 19: /R~{CS} -> /Q3
- U2 pad 2: /RD3 -> /D7
- U2 pad 3: /RD2 -> /D6
- U2 pad 4: /RD4 -> /D5
- U2 pad 5: /RD7 -> /D4
- U2 pad 6: /RD0 -> /D3
- U2 pad 7: /RD6 -> /D2
- U2 pad 8: /RD1 -> /D1
- U2 pad 9: /RD5 -> /D0
- U7 pad 11: unconnected-(U7-Pad11) -> /DDIR
- U7 pad 12: /R~{W} -> /~{R}W
- U7 pad 13: /A13 -> /R~{CS}
- U9 pad 11: Net-(U10-Pad9) -> unconnected-(U9-Pad11)
Routing:
- net /DDIR: track 0.00 -> 46.3 mm, vias 0 -> 2
- net /Q3: track 0.00 -> 44.7 mm, vias 0 -> 5
- net /R~{CS}: track 79.0 -> 108.2 mm
- net /~{R}W: track 13.5 -> 38.4 mm
- net Net-(U10-Pad9): track 11.7 -> 0.00 mm
- net (no net): track 0.00 -> 11.7 mm
- net /R~{W}: track 87.2 -> 77.5 mm, vias 6 -> 4
- net /RCS: track 112.2 -> 107.3 mm
- net /DMAin: track 123.0 -> 118.4 mm
- net /RA12: track 74.2 -> 69.6 mm
- net /RD4: track 11.3 -> 15.5 mm
- net Net-(R4-Pad2): track 48.4 -> 44.4 mm
- net /RD2: track 26.1 -> 30.0 mm
- net /RD3: track 14.0 -> 17.6 mm
- net +5V: track 88.1 -> 90.2 mm, vias 74 -> 75
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Other:
- board text added: "B12"
- board text removed: "B11"

Commit message: 1.2?
Connections:
- U10 pad 9: unconnected-(U10-Pad9) -> Net-(U10-Pad9)
- U9 pad 11: unconnected-(U9-Pad11) -> Net-(U10-Pad9)
Routing:
- net Net-(U10-Pad9): track 0.00 -> 11.7 mm
- net (no net): track 11.7 -> 0.00 mm
- net /RCS: track 107.3 -> 106.6 mm
