File: RAM128.kicad_pcb (KiCad board)
At the start: 4 copper layers, 74.2 x 42.7 mm, 57 parts, among them J1 AppleIIBus, SW1 DMA/ROM, U1 621024, U10 74AHCT32PW, U11 74AHCT1G126GW, U12 74AHCT1G04GW, U13 74AHCT1G04GW, U14 74AHCT1G04GW, U15 74AHCT1G04GW, U16 74AHCT1G04GW, U17 74AHCT1G04GW, U18 74AHCT1G32GW, U19 74AHCT1G04GW, U2 74HCT245PW, U20 74AHCT1G04GW, U3 74HCT273PW, U4 74HCT273PW, U5 74AHCT1G32GW, U6 74AHCT08PW, U7 74AHCT32PW, U8 74AHCT08PW, U9 74AHCT08PW

Commit message: RC 1.3
Other:
- board text added: "B13"
- board text removed: "B12"
Changed lines of the file:
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@@
   (title_block
     (title "RAM128 (GW4208B)")
-    (date "2023-12-07")
-    (rev "1.2")
+    (date "2024-03-29")
+    (rev "1.3")
     (company "Garrett's Workshop")
   )
@@
     (property "ki_description" "Generic connector, double row, 02x25, counter clockwise pin numbering scheme (similar to DIP packge numbering), script generated (kicad-library-utils/schlib/autogen/connector/)")
     (property "ki_keywords" "connector")
-    (attr exclude_from_pos_files exclude_from_bom allow_soldermask_bridges)
+    (attr exclude_from_pos_files allow_soldermask_bridges)
     (fp_text reference "J1" (at 0 4.953) (layer "F.Fab")
         (effects (font (size 0.8128 0.8128) (thickness 0.2032)))
@@
     (at 106.05 127.85)
     (tags "SOT-353 SC-70-5")
+    (property "LCSC Part" "C554582")
     (property "Sheetfile" "RAM128.kicad_sch")
     (property "Sheetname" "")
@@
     (at 103.05 127.85)
     (tags "SOT-353 SC-70-5")
+    (property "LCSC Part" "C554582")
     (property "Sheetfile" "RAM128.kicad_sch")
     (property "Sheetname" "")
@@
     (effects (font (size 0.8128 0.8128) (thickness 0.2032) bold) (justify mirror))
   )
-  (gr_text "B12" (at 73.0885 130.302) (layer "B.SilkS")
+  (gr_text "B13" (at 73.0885 130.302) (layer "B.SilkS")
     (effects (font (size 0.8128 0.8128) (thickness 0.2032) bold) (justify mirror))
   )

Commit message: idk
Parts:
- added C20: 2u2, stdpads:C_0603, F.Cu at (58.6, 114.9)
- added D1: Amber, stdpads:LED_0805, F.Cu at (35.9, 102.4)
- added D2: Amber, stdpads:LED_0805, F.Cu at (35.9, 105.5)
- added D3: Amber, stdpads:LED_0805, F.Cu at (35.9, 108.5)
- added D4: Amber, stdpads:LED_0805, F.Cu at (35.9, 111.5)
- added D5: Amber, stdpads:LED_0805, F.Cu at (35.9, 114.5)
- added D6: Amber, stdpads:LED_0805, F.Cu at (35.9, 117.5)
- added R10: 22k, stdpads:R_0805, F.Cu at (40.3, 111.6)
- added R11: 470, stdpads:R_0805, F.Cu at (40.3, 114.7)
- added R12: 470, stdpads:R_0805, F.Cu at (44.8, 102.5)
- added R13: 470, stdpads:R_0805, F.Cu at (44.8, 105.5)
- added R14: 470, stdpads:R_0805, F.Cu at (44.8, 108.6)
- added R15: 470, stdpads:R_0805, F.Cu at (44.8, 111.6)
- added R16: 470, stdpads:R_0805, F.Cu at (44.8, 114.7)
- added R7: 22k, stdpads:R_0805, F.Cu at (40.3, 102.5)
- added R8: 22k, stdpads:R_0805, F.Cu at (40.3, 105.5)
- added R9: 22k, stdpads:R_0805, F.Cu at (40.3, 108.6)
- added U21: 74AHCT1G04GW, stdpads:SOT-353, F.Cu at (48.8, 103.1)
- added U22: 74AHCT1G04GW, stdpads:SOT-353, F.Cu at (52.5, 103.1)
- added U23: 74AHCT1G04GW, stdpads:SOT-353, F.Cu at (56.1, 103.1)
- added U24: 74AHCT1G32GW, stdpads:SOT-353, F.Cu at (59.8, 103.1)
- added U25: 74AHCT1G04GW, stdpads:SOT-353, F.Cu at (48.8, 107.3)
- added U26: 74AHCT1G08GW, stdpads:SOT-353, F.Cu at (52.5, 107.3)
- added U27: 74AHCT1G08GW, stdpads:SOT-353, F.Cu at (56.1, 107.3)
- added U28: 74AHCT1G08GW, stdpads:SOT-353, F.Cu at (59.8, 107.3)
- added U29: 74AHCT1G08GW, stdpads:SOT-353, F.Cu at (48.8, 111.6)
- added U30: 74AHCT1G08GW, stdpads:SOT-353, F.Cu at (52.5, 111.6)
- added U31: 74AHCT1G08GW, stdpads:SOT-353, F.Cu at (56.1, 111.6)
- H1, H2, H3, H4, H5: value (none) -> ~
- SW1: value DMA/ROM -> CFG; footprint stdpads:SW_DIP_SPSTx02_Slide_DSHP02TS_P1.27mm -> stdpads:SW_DIP_SPSTx05_Slide_DSHP05TS_P1.27mm
- moved SW1 19.7 mm to (51.9, 119.0)
Connections:
- R2 pad 1: Net-(R2-Pad1) -> /RCSsw
- R4 pad 2: Net-(R4-Pad2) -> /DMAinsw
- SW1 pad 1: Net-(R4-Pad2) -> /DMAin
- SW1 pad 2: Net-(R2-Pad1) -> /RCS
- SW1 pad 3: /RCS -> /~{A2}
- SW1 pad 4: /DMAin -> /RES
- U3 pad 1: /~{RES} -> /~{RRST}
- U4 pad 1: /~{RES} -> /~{RRST}
- U6 pad 13: Net-(R4-Pad2) -> /DMAinsw
- U7 pad 4: /A2 -> /BA2
- U7 pad 9: Net-(R2-Pad1) -> /RCSsw
Routing:
- net Net-(R4-Pad2): track 43.9 -> 0.00 mm, vias 2 -> 0
- net /DMAinsw: track 0.00 -> 43.9 mm, vias 0 -> 2
- net Net-(R2-Pad1): track 42.7 -> 0.00 mm, vias 2 -> 0
- net /RCSsw: track 0.00 -> 42.7 mm, vias 0 -> 2
Other:
- board text added: "C10"
- board text removed: "B13"

Commit message: schematic and placement done?
Parts:
- removed the G*** at (108.0, 100.9)
- removed the G*** at (125.6, 100.8)
- removed U16, U17, U19, U20, U21, U22, U23, U25: 74AHCT1G04GW, stdpads:SOT-353
- removed U24: 74AHCT1G32GW, stdpads:SOT-353
- removed U26, U27, U28, U29, U30, U31: 74AHCT1G08GW, stdpads:SOT-353
- added C19: 2u2, stdpads:C_0603, F.Cu at (117.2, 93.7)
- added C21: 2u2, stdpads:C_0603, F.Cu at (130.8, 123.3)
- added FID5: Fiducial, stdpads:Fiducial, F.Cu at (48.1, 129.5)
- added G***: LOGO, LOGO, F.Cu at (112.9, 83.9)
- added G***: LOGO, LOGO, F.Cu at (91.4, 84.0)
- added Q1: MMBT3904, stdpads:SOT-23, F.Cu at (142.8, 123.6)
- added R17: 470, stdpads:R_0805, F.Cu at (56.1, 98.7)
- C16: value 10u -> 2u2; footprint stdpads:C_0805 -> stdpads:C_0603
- C2, C3, C4, C5: value 2u2 -> 10u; footprint stdpads:C_0603 -> stdpads:C_0805
- R1, R10, R3, R7, R8, R9: value 22k -> 10k; footprint stdpads:R_0805 -> stdpads:R_0603
- R11: value 470 -> 10k; footprint stdpads:R_0805 -> stdpads:R_0603
- R2: value 22k -> 2k2; footprint stdpads:R_0805 -> stdpads:R_0603
- R4: value 22k -> 47; footprint stdpads:R_0805 -> stdpads:R_0603
- R5: value 0 -> 10k; footprint stdpads:R_0805 -> stdpads:R_0603
- R6: value DNP -> 10k; footprint stdpads:R_0805 -> stdpads:R_0603
- U10: value 74AHCT32PW -> 74AHC1G14GW; footprint stdpads:TSSOP-14_4.4x5mm_P0.65mm -> stdpads:SOT-353
- U11: value 74AHCT1G126GW -> 74AHCT08PW; footprint stdpads:SOT-353 -> stdpads:TSSOP-14_4.4x5mm_P0.65mm
- U12, U13: value 74AHCT1G04GW -> 74AHCT32PW; footprint stdpads:SOT-353 -> stdpads:TSSOP-14_4.4x5mm_P0.65mm
- U14: value 74AHCT1G04GW -> 74AHCT1G125GW
- U15: value 74AHCT1G04GW -> 74AHC1G14GW
- U18, U5: value 74AHCT1G32GW -> 74HCT273PW; footprint stdpads:SOT-353 -> stdpads:TSSOP-20_4.4x6.5mm_P0.65mm
- U3: value 74HCT273PW -> 74AHCT00PW; footprint stdpads:TSSOP-20_4.4x6.5mm_P0.65mm -> stdpads:TSSOP-14_4.4x5mm_P0.65mm
- U4: value 74HCT273PW -> 74AHC1G14GW; footprint stdpads:TSSOP-20_4.4x6.5mm_P0.65mm -> stdpads:SOT-353
- U6: value 74AHCT08PW -> 74AHCT02PW
- U7: value 74AHCT32PW -> 74AHCT08PW
- moved H2 88.9 mm to (48.1, 127.0), turned to 0 degrees
- moved FID1 88.7 mm to (143.0, 82.4), turned to -90 degrees
- moved SW1 86.7 mm to (134.7, 93.3)
- moved R1 82.0 mm to (51.2, 122.3), turned to 90 degrees
- moved FID3 80.9 mm to (58.8, 82.9), turned to 90 degrees
- moved C20 77.2 mm to (135.3, 123.3), turned to -90 degrees
- moved R11 75.1 mm to (113.2, 96.2), turned to 180 degrees
- moved R10 74.1 mm to (113.2, 97.7), turned to 180 degrees
- moved R8 73.9 mm to (113.2, 93.2), turned to 180 degrees
- moved R9 73.4 mm to (113.2, 99.2), turned to 180 degrees
- moved R7 73.2 mm to (113.2, 94.7)
- moved C6 72.5 mm to (52.8, 122.3)
- moved H1 70.1 mm to (140.5, 129.5)
- moved U4 57.4 mm to (55.4, 121.6)
- moved C9 46.3 mm to (55.5, 119.2), turned to 180 degrees
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Connections:
- net /7M renamed /Bus/7M
- net /COLORREF renamed /Bus/COLORREF
- net /DMA renamed /Bus/~{DMA}
- net /INTin renamed /Bus/INTin
- net /RDY renamed /Bus/RDY
- net /USER1 renamed /Bus/USER1
- net /VIDSYNC renamed /Bus/VIDSYNC
- net /~{IOSEL} renamed /Bus/~{IOSEL}
- net /~{IOSTRB} renamed /Bus/~{IOSTRB}
- net /~{IRQ} renamed /Bus/~{IRQ}
- net /~{NMI} renamed /Bus/~{NMI}
- C16 pad 1: +12V -> +5V
- C2 pad 1: +5V -> -12V
- C20 pad 1: /~{PUP} -> +5V
- C3 pad 1: +5V -> +12V
- C4 pad 1: +5V -> -5V
- C6 pad 1: +5V -> /Control/~{POR}
- D1 pad 2: /LED_RA16 -> /LEDs/LED_RA16
- D2 pad 2: /LED_RA15 -> /LEDs/LED_RA15
- D3 pad 2: /LED_RA14 -> /LEDs/LED_RA14
- D4 pad 2: /LED_ENRD -> /LEDs/LED_ENRD
- D5 pad 2: /LED_ENWR -> /LEDs/LED_ENWR
- D6 pad 2: /LED_ACT -> /LEDs/LED_ACT
- J1 pad 10: /A8 -> /Bus/A8
- J1 pad 11: /A9 -> /Bus/A9
- J1 pad 12: /A10 -> /Bus/A10
- J1 pad 13: /A11 -> /Bus/A11
- J1 pad 14: /A12 -> /Bus/A12
- J1 pad 15: /A13 -> /Bus/A13
- J1 pad 16: /A14 -> /Bus/A14
- J1 pad 17: /A15 -> /Bus/A15
- J1 pad 18: /R~{W} -> /Control/R~{W}
- J1 pad 2: /A0 -> /Bus/A0
- J1 pad 24: /DMAout -> /Bus/DMAout
- J1 pad 27: /DMAin -> /Control/DMAin
- J1 pad 3: /A1 -> /Bus/A1
- J1 pad 31: /~{RES} -> /Control/~{RESET}
- J1 pad 32: /~{INH} -> /Buf/~{INH}
- J1 pad 37: /Q3 -> /Bus/Q3
- J1 pad 38: /PHI1 -> /Control/PHI1
- J1 pad 4: /A2 -> /Bus/A2
- J1 pad 40: /PHI0 -> /Bus/PHI0
- J1 pad 41: /~{DEVSEL} -> /Bus/~{DEVSEL}
- J1 pad 42: /D7 -> /Buf/D7
- J1 pad 43: /D6 -> /Buf/D6
- J1 pad 44: /D5 -> /Buf/D5
- J1 pad 45: /D4 -> /Buf/D4
- J1 pad 46: /D3 -> /Buf/D3
- J1 pad 47: /D2 -> /Buf/D2
- J1 pad 48: /D1 -> /Buf/D1
- J1 pad 49: /D0 -> /Buf/D0
- J1 pad 5: /A3 -> /Bus/A3
- J1 pad 6: /A4 -> /Bus/A4
- J1 pad 7: /A5 -> /Bus/A5
- J1 pad 8: /A6 -> /Bus/A6
- J1 pad 9: /A7 -> /Bus/A7
- R1 pad 2: /~{INH} -> /Control/~{POR}
- R10 pad 2: /~{PUP} -> Net-(R10-Pad2)
- R11 pad 1: /LED_RA16 -> +5V
- R11 pad 2: Net-(U26-Y) -> Net-(R11-Pad2)
- R12 pad 1: /LED_RA15 -> /LEDs/LED_RA16
- R12 pad 2: Net-(U27-Y) -> Net-(R12-Pad2)
- R13 pad 1: /LED_RA14 -> /LEDs/LED_RA15
- R13 pad 2: Net-(U28-Y) -> Net-(R13-Pad2)
- R14 pad 1: /LED_ENRD -> /LEDs/LED_RA14
- R14 pad 2: Net-(U29-Y) -> Net-(R14-Pad2)
- R15 pad 1: /LED_ENWR -> /LEDs/LED_ENRD
- R15 pad 2: Net-(U30-Y) -> Net-(R15-Pad2)
- R16 pad 1: /LED_ACT -> /LEDs/LED_ENWR
- R16 pad 2: Net-(U31-Y) -> Net-(R16-Pad2)
- R2 pad 1: /RCSsw -> /Control/POR
- R2 pad 2: GND -> Net-(Q1-B)
- R3 pad 1: +5V -> Net-(Q1-B)
- R3 pad 2: /DMAin -> GND
- R4 pad 1: +5V -> /Control/~{RESET}
- R4 pad 2: /DMAinsw -> Net-(Q1-C)
- R5 pad 1: /~{INH} -> +5V
- R5 pad 2: Net-(U11-Y) -> /Buf/~{INH}
- R6 pad 1: /R~{W} -> +5V
- R6 pad 2: /R~{WE} -> /Control/DMAin
- R7 pad 1: /LEDEN -> /Config/DMAoutEN
- R8 pad 1: /RESsw -> /Config/LEDEN
- R9 pad 2: Net-(R9-Pad2) -> /Config/DMAinsw
- SW1 pad 1: /DMAin -> /Control/DMAin
- SW1 pad 10: /DMAinsw -> /Config/DMAinsw
- SW1 pad 2: /RCS -> /Config/DMAoutEN
- SW1 pad 3: /~{A2} -> /Bus/A2
- SW1 pad 4: /RES -> /Config/RES
- SW1 pad 5: /LEDEN -> /Config/LEDEN
- SW1 pad 6: Net-(R9-Pad2) -> Net-(R11-Pad2)
- SW1 pad 7: /RESsw -> /Config/RESsw
- SW1 pad 8: /~{A2}sw -> /Config/A2sw
- SW1 pad 9: /RCSsw -> Net-(R10-Pad2)
- U1 pad 10: /A3 -> /LEDs/RA15
- U1 pad 11: /A2 -> /LEDs/RA14
- U1 pad 12: /A0 -> /Control/RA12
- U1 pad 13: /RD0 -> /Buf/RD0
- U1 pad 14: /RD1 -> /Buf/RD1
- U1 pad 15: /RD2 -> /Buf/RD2
- U1 pad 17: /RD3 -> /Buf/RD3
- U1 pad 18: /RD4 -> /Buf/RD4
- U1 pad 19: /RD5 -> /Buf/RD5
- U1 pad 2: /RA16 -> /Bus/A13
- U1 pad 20: /RD6 -> /Buf/RD6
- U1 pad 21: /RD7 -> /Buf/RD7
- U1 pad 22: /R~{CS} -> GND
- U1 pad 23: /A1 -> /Bus/A8
- U1 pad 24: /~{R}W -> /Control/~{R}W
- U1 pad 25: /A4 -> /Bus/A0
- U1 pad 26: /A6 -> /Bus/A2
- U1 pad 27: /A8 -> /Bus/A4
- U1 pad 28: /A10 -> /Bus/A6
- U1 pad 29: /R~{WE} -> /Control/R~{WE}
- U1 pad 3: /RA15 -> /Bus/A11
- U1 pad 30: +5V -> /Control/RCS
- U1 pad 31: /A13 -> /Bus/A10
- U1 pad 4: /RA14 -> /Bus/A9
- U1 pad 5: /RA12 -> /Bus/A7
- U1 pad 6: /A11 -> /Bus/A5
- U1 pad 7: /A9 -> /Bus/A3
- U1 pad 8: /A7 -> /Bus/A1
- U1 pad 9: /A5 -> /LEDs/RA16
- U10 pad 1: Net-(U10-Pad1) -> unconnected-(U10-NC-Pad1)
- U10 pad 2: Net-(U10-Pad2) -> /Control/R~{W}
- U10 pad 3: /~{A0XOR1} -> GND
- U10 pad 4: Net-(U10-Pad4) -> /Control/~{R}W
- U10 pad 5: Net-(U10-Pad5) -> +5V
- U11 pad 1: /INHOE -> /Bus/A12
- U11 pad 2: GND -> /Bus/A13
- U11 pad 3: GND -> Net-(U11-Pad3)
- U11 pad 4: Net-(U11-Y) -> /Control/R~{W}
- U11 pad 5: +5V -> /Control/RCS
- U12 pad 1: unconnected-(U12-NC-Pad1) -> /Bus/Q3
- U12 pad 2: /A2 -> /Control/PHI1
- U12 pad 3: GND -> /Control/D~{OE}
- U12 pad 4: /~{A2} -> /Control/D~{OE}
- U12 pad 5: +5V -> /Control/R~{W}
- U13 pad 1: unconnected-(U13-NC-Pad1) -> Net-(U11-Pad8)
- U13 pad 2: /A0 -> Net-(U13-Pad2)
- U13 pad 3: GND -> Net-(U13-Pad3)
- U13 pad 4: /~{A0} -> /Control/~{A2}
- U13 pad 5: +5V -> /Bus/~{DEVSEL}
- U14 pad 1: unconnected-(U14-NC-Pad1) -> /Buf/INH~{OE}
- U14 pad 2: /A1 -> GND
- U14 pad 4: /~{A1} -> /Buf/~{INH}
- U15 pad 2: /A13 -> /Control/~{RESET}
- U15 pad 4: /~{A13} -> /Config/RES
- U18 pad 1: /R~{W} -> /Control/R~{RST}
- U18 pad 2: /D~{OE} -> /Control/BankAB
- U18 pad 3: GND -> /Bus/A3
- U18 pad 4: /R~{WE} -> /Control/~{A0XOR1}
- U18 pad 5: +5V -> /Control/ENRD
- U2 pad 1: /DDIR -> /Buf/DDIR
- U2 pad 11: /RD3 -> /Buf/D0
- U2 pad 12: /RD2 -> /Buf/D1
- U2 pad 13: /RD4 -> /Buf/D2
- U2 pad 14: /RD7 -> /Buf/D3
- U2 pad 15: /RD0 -> /Buf/D4
- U2 pad 16: /RD6 -> /Buf/D5
- U2 pad 17: /RD1 -> /Buf/D6
- U2 pad 18: /RD5 -> /Buf/D7
- U2 pad 19: /D~{OE} -> /Control/D~{OE}
- U2 pad 2: /D7 -> /Buf/RD5
- U2 pad 3: /D6 -> /Buf/RD1
- U2 pad 4: /D5 -> /Buf/RD6
- U2 pad 5: /D4 -> /Buf/RD0
- U2 pad 6: /D3 -> /Buf/RD7
- U2 pad 7: /D2 -> /Buf/RD4
- U2 pad 8: /D1 -> /Buf/RD2
- U2 pad 9: /D0 -> /Buf/RD3
- U3 pad 1: /~{RRST} -> /Bus/A2
- U3 pad 10: GND -> /Config/DMAinsw
- U3 pad 11: /~{A2}clk -> Net-(U11-Pad12)
- U3 pad 12: unconnected-(U3-Q4-Pad12) -> /Control/RCS
- U3 pad 13: GND -> /Config/DMAoutEN
- U3 pad 14: GND -> +5V
- U3 pad 2: /BankAB -> +5V
- U3 pad 3: /A3 -> /Control/~{A2}
- U3 pad 4: /~{A0XOR1} -> Net-(U13-Pad3)
- U3 pad 5: /ENRD -> Net-(U3-Pad5)
- U3 pad 6: /ENWR1 -> /Buf/INH~{OE}
- U3 pad 7: /A0 -> GND
- U3 pad 8: /ENWR1A0 -> Net-(U3-Pad8)
- U3 pad 9: /ENWR -> /Control/INH
- U4 pad 1: /~{RRST} -> unconnected-(U4-NC-Pad1)
- U4 pad 2: /RA16 -> /Control/~{POR}
- U4 pad 3: /A3 -> GND
- U4 pad 4: /A1 -> /Control/POR
- U4 pad 5: /RA15 -> +5V
- U5 pad 1: /PHI1 -> /Control/R~{RST}
- U5 pad 2: /Q3 -> /LEDs/RA16
- U5 pad 3: GND -> /Bus/A3
- U5 pad 4: /D~{OE} -> /Bus/A1
- U5 pad 5: +5V -> /LEDs/RA15
- U6 pad 1: /~{A0} -> Net-(U12-Pad9)
- U6 pad 10: /A0 -> /Control/R~{RST}
- U6 pad 11: Net-(U6-Pad11) -> Net-(U3-Pad8)
- U6 pad 12: /INHOE -> /Control/PHI1
- U6 pad 13: /DMAinsw -> /Control/RCS
- U6 pad 2: /~{A1} -> /Bus/A13
- U6 pad 3: Net-(U10-Pad1) -> /Control/BankAB
- U6 pad 4: /A0 -> Net-(U13-Pad9)
- U6 pad 5: /A1 -> /Bus/A0
- U6 pad 6: Net-(U10-Pad2) -> /Bus/A1
- U6 pad 8: /ENWR1A0 -> /Control/POR
- U6 pad 9: /ENWR1 -> /Config/RESsw
- U7 pad 1: /~{A2} -> /Control/ENWR
- U7 pad 10: Net-(U19-Y) -> /Config/LEDEN
- U7 pad 11: /DDIR -> Net-(R17-Pad2)
- U7 pad 12: /~{R}W -> /Control/RCS
- U7 pad 13: /R~{CS} -> /Config/LEDEN
- U7 pad 2: /~{DEVSEL} -> /Control/~{R}W
- U7 pad 3: /A2clk -> Net-(U13-Pad2)
- U7 pad 4: /BA2 -> Net-(U7-Pad4)
- U7 pad 5: /~{DEVSEL} -> Net-(U12-Pad11)
- U7 pad 6: /~{A2}clk -> Net-(U3-Pad5)
- U7 pad 8: /~{DMAout} -> Net-(R16-Pad2)
- U7 pad 9: /RCSsw -> /Control/ENWR
- U8 pad 1: /A12 -> /LEDs/RA16
- U8 pad 10: /~{R}W -> /Config/LEDEN
- U8 pad 11: Net-(U8-Pad11) -> Net-(R15-Pad2)
- U8 pad 12: /A15 -> /Control/ENRD
- U8 pad 13: /A14 -> /Config/LEDEN
- U8 pad 2: /A13 -> /Config/LEDEN
- U8 pad 3: Net-(U10-Pad5) -> Net-(R12-Pad2)
- U8 pad 4: /~{A13} -> /LEDs/RA15
- U8 pad 5: /BankAB -> /Config/LEDEN
- U8 pad 6: Net-(U10-Pad4) -> Net-(R13-Pad2)
- U8 pad 8: Net-(U10-Pad10) -> Net-(R14-Pad2)
- U8 pad 9: /ENWR -> /LEDs/RA14
- U9 pad 1: Net-(U8-Pad11) -> /Bus/A1
- U9 pad 10: Net-(U9-Pad10) -> Net-(U3-Pad5)
- U9 pad 11: Net-(U10-Pad9) -> Net-(U7-Pad4)
- U9 pad 12: /ENRD -> /Bus/A15
- U9 pad 13: /R~{W} -> /Bus/A14
- U9 pad 2: Net-(U10-Pad11) -> /Bus/A0
- U9 pad 3: Net-(U9-Pad10) -> Net-(U13-Pad10)
- U9 pad 4: Net-(U6-Pad11) -> /Control/ENWR1
- U9 pad 5: /PHI0 -> /Bus/A0
- U9 pad 6: /RCS -> /Control/ENWR1A0
- U9 pad 8: /INHOE -> /Control/INH
- U9 pad 9: Net-(U10-Pad8) -> Net-(U13-Pad3)
Routing:
- net /A0: track 128.2 -> 0.00 mm, vias 5 -> 0
- net /DMAin: track 119.3 -> 0.00 mm, vias 4 -> 0
- net /RCS: track 106.7 -> 0.00 mm, vias 6 -> 0
- net /R~{CS}: track 106.4 -> 0.00 mm, vias 3 -> 0
- net /A1: track 102.0 -> 0.00 mm, vias 3 -> 0
- net /A3: track 89.0 -> 0.00 mm, vias 2 -> 0
- net /A13: track 70.1 -> 0.00 mm, vias 4 -> 0
- net /RA12: track 69.6 -> 0.00 mm, vias 4 -> 0
- net /~{RES}: track 68.6 -> 0.00 mm, vias 2 -> 0
- net /~{R}W: track 58.3 -> 0.00 mm, vias 2 -> 0
- net /R~{W}: track 54.3 -> 0.00 mm, vias 4 -> 0
- net /A2: track 53.6 -> 0.00 mm, vias 3 -> 0
- net /INHOE: track 53.6 -> 0.00 mm, vias 4 -> 0
- net /A11: track 47.0 -> 0.00 mm
- net /DDIR: track 46.3 -> 0.00 mm, vias 2 -> 0
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- added copper zone on In2.Cu, net /Buf/DDIR
- removed copper zone on In2.Cu, net +5V
Other:
- board size 74.2 x 42.7 mm -> 99.9 x 59.8 mm
- board text added: "1"
- board text added: "128 kB capacity"
- board text added: "16 kB capacity"
- board text added: "2"
- board text added: "4"
- board text added: "Activity"
- board text added: "Bank"
- board text added: "LEDs disabled"
- board text added: "LEDs enabled"
- board text added: "ROM sharing off"
- board text added: "ROM sharing on"
- board text added: "Read Enabled"
- board text added: "Reset disabled"
- board text added: "Reset enabled"
- board text added: "Write Enabled"
- board text removed: "DMA/ROM control"
- board text removed: "JLCJLCJLCJLC"
- board text removed: "in"
- board text removed: "out"

Commit message: more
Parts:
- moved D2 23.5 mm to (76.0, 82.7)
- moved D3 23.5 mm to (78.2, 82.7)
- moved R12 23.5 mm to (78.2, 86.1)
- moved R17 23.5 mm to (76.0, 86.1)
- moved D1 23.5 mm to (73.8, 82.7)
- moved R16 23.5 mm to (73.8, 86.1)
- moved D5 13.7 mm to (70.3, 82.7)
- moved R14 13.7 mm to (70.3, 86.1)
- moved D4 13.6 mm to (66.8, 82.7)
- moved R13 13.6 mm to (66.8, 86.1)
- moved D6 13.3 mm to (63.3, 82.8)
- moved R15 13.3 mm to (63.3, 86.2)
- moved C5 6.50 mm to (95.6, 107.4)
- moved U1 1.78 mm to (84.1, 101.6)
- turned C2 to 0 degrees
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Connections:
- C3 pad 1: +12V -> -5V
- C4 pad 1: -5V -> +12V
- U1 pad 13: /Buf/RD0 -> /Buf/RD5
- U1 pad 14: /Buf/RD1 -> /Buf/RD3
- U1 pad 15: /Buf/RD2 -> /Buf/RD1
- U1 pad 17: /Buf/RD3 -> /Buf/RD0
- U1 pad 18: /Buf/RD4 -> /Buf/RD2
- U1 pad 19: /Buf/RD5 -> /Buf/RD4
- U1 pad 2: /Bus/A13 -> /Bus/A11
- U1 pad 23: /Bus/A8 -> /Bus/A0
- U1 pad 25: /Bus/A0 -> /Bus/A3
- U1 pad 26: /Bus/A2 -> /Bus/A5
- U1 pad 27: /Bus/A4 -> /Bus/A7
- U1 pad 28: /Bus/A6 -> /Bus/A9
- U1 pad 3: /Bus/A11 -> /Bus/A10
- U1 pad 31: /Bus/A10 -> /Bus/A13
- U1 pad 4: /Bus/A9 -> /Bus/A8
- U1 pad 5: /Bus/A7 -> /Bus/A6
- U1 pad 6: /Bus/A5 -> /Bus/A4
- U1 pad 7: /Bus/A3 -> /Bus/A2
- U2 pad 2: /Buf/RD5 -> /Buf/RD7
- U2 pad 3: /Buf/RD1 -> /Buf/RD6
- U2 pad 4: /Buf/RD6 -> /Buf/RD5
- U2 pad 5: /Buf/RD0 -> /Buf/RD4
- U2 pad 6: /Buf/RD7 -> /Buf/RD3
- U2 pad 7: /Buf/RD4 -> /Buf/RD2
- U2 pad 8: /Buf/RD2 -> /Buf/RD1
- U2 pad 9: /Buf/RD3 -> /Buf/RD0
Routing:
- net /Control/PHI1: track 0.00 -> 55.9 mm, vias 0 -> 2
- net /Bus/A13: track 34.2 -> 84.5 mm, vias 0 -> 4
- net /Bus/A2: track 21.6 -> 63.9 mm, vias 0 -> 2
- net /Control/R~{W}: track 9.31 -> 47.4 mm
- net /Bus/A12: track 4.61 -> 38.1 mm
- net /Bus/A5: track 0.00 -> 29.3 mm
- net /Bus/A4: track 17.9 -> 43.1 mm
- net /Bus/A6: track 19.4 -> 44.2 mm
- net /Bus/A8: track 23.5 -> 48.2 mm
- net /Bus/A10: track 26.7 -> 51.4 mm
- net /Buf/RD1: track 0.00 -> 24.3 mm
- net /Buf/RD5: track 0.00 -> 24.3 mm
- net /Buf/RD3: track 0.00 -> 24.3 mm
- net /Bus/A11: track 29.2 -> 53.2 mm
- net /Bus/A14: track 9.27 -> 30.8 mm, vias 0 -> 2
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Other:
- board text added: "ACT"
- board text added: "RD"
- board text added: "WR"
- board text removed: "Activity"
- board text removed: "Read Enabled"
- board text removed: "Write Enabled"

Commit message: more
Parts:
- moved C21 6.70 mm to (137.5, 123.5), turned to 90 degrees
- moved U10 6.40 mm to (131.1, 123.4), turned to 180 degrees
- moved U15 2.45 mm to (135.3, 123.4), turned to 180 degrees
- moved C20 2.16 mm to (133.2, 123.5), turned to 90 degrees
- moved C8 0.10 mm to (128.9, 123.5)
- renumbered U15 to U10, U10 to U15
Connections:
- U10 pad 2: /Control/~{RESET} -> /Control/R~{W}
- U10 pad 4: /Config/RES -> /Control/~{R}W
- U12 pad 10: Net-(U11-Pad3) -> /Bus/A13
- U12 pad 11: Net-(U12-Pad11) -> /Control/RA12
- U12 pad 12: /Bus/A13 -> Net-(U11-Pad3)
- U12 pad 13: /Bus/A12 -> Net-(U12-Pad13)
- U12 pad 8: /Control/RA12 -> Net-(U12-Pad8)
- U12 pad 9: Net-(U12-Pad9) -> /Bus/A12
- U15 pad 2: /Control/R~{W} -> /Control/~{RESET}
- U15 pad 4: /Control/~{R}W -> /Config/RES
- U6 pad 1: Net-(U12-Pad9) -> Net-(U12-Pad13)
- U7 pad 5: Net-(U12-Pad11) -> Net-(U12-Pad8)
- U9 pad 10: Net-(U3-Pad5) -> /Bus/A14
- U9 pad 11: Net-(U7-Pad4) -> /Control/INH
- U9 pad 12: /Bus/A15 -> Net-(U3-Pad5)
- U9 pad 13: /Bus/A14 -> Net-(U13-Pad3)
- U9 pad 8: /Control/INH -> Net-(U7-Pad4)
- U9 pad 9: Net-(U13-Pad3) -> /Bus/A15
Routing:
- net /Control/RCS: track 0.00 -> 54.6 mm, vias 0 -> 4
- net /Control/D~{OE}: track 2.73 -> 49.8 mm, vias 1 -> 2
- net Net-(U12-Pad13): track 0.00 -> 45.2 mm, vias 0 -> 2
- net /Buf/DDIR: track 0.00 -> 41.3 mm, vias 0 -> 2
- net Net-(U3-Pad8): track 0.00 -> 25.7 mm, vias 0 -> 2
- net /Buf/INH~{OE}: track 0.00 -> 24.6 mm, vias 0 -> 2
- net Net-(U11-Pad3): track 0.00 -> 24.2 mm
- net /Control/POR: track 2.15 -> 24.9 mm
- net /Bus/~{DEVSEL}: track 12.4 -> 31.0 mm, vias 2 -> 1
- net Net-(U13-Pad3): track 0.00 -> 14.4 mm
- net Net-(U3-Pad5): track 0.00 -> 14.1 mm
- net GND: track 70.9 -> 85.0 mm, vias 166 -> 179
- net /Control/INH: track 0.00 -> 13.0 mm, vias 0 -> 2
- net +5V: track 100.2 -> 112.0 mm, vias 65 -> 76
- net Net-(U13-Pad10): track 0.00 -> 11.2 mm, vias 0 -> 2
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- added copper zone on In2.Cu, net +5V
- removed copper zone on In2.Cu, net /Buf/DDIR
