File: Buf.kicad_sch (KiCad schematic)
At the start: 3 parts, among them U11 74AHCT1G125GW, U2 74HCT245PW

Commit message: schematic and placement done?
Parts:
- removed U11: 74AHCT1G125GW, stdpads:SOT-353, symbol GW_Logic:741G125GW
- added C7, C8: 2u2, stdpads:C_0603, symbol Device:C_Small
- added U14: 74AHCT1G125GW, stdpads:SOT-353, symbol GW_Logic:741G125GW
- R5: value 22k -> 10k; footprint stdpads:R_0805 -> stdpads:R_0603
Connections:
- net +5V: now also C7.1, C8.1, U14.5 (Vcc)
- net D0: now also U2.11 (B7); no longer U2.9 (A7)
- net D1: now also U2.12 (B6); no longer U2.8 (A6)
- net D2: now also U2.13 (B5); no longer U2.7 (A5)
- net D3: now also U2.14 (B4); no longer U2.6 (A4)
- net D4: now also U2.15 (B3); no longer U2.5 (A3)
- net D5: now also U2.16 (B2); no longer U2.4 (A2)
- net D6: now also U2.17 (B1); no longer U2.3 (A1)
- net D7: now also U2.18 (B0); no longer U2.2 (A0)
- net GND: now also C7.2, C8.2, U14.2 (A), U14.3 (GND)
- net INH~{OE}: now also U14.1 (~{OE})
- net RD0: now also U2.5 (A3); no longer U2.15 (B3)
- net RD1: now also U2.3 (A1); no longer U2.17 (B1)
- net RD2: now also U2.8 (A6); no longer U2.12 (B6)
- net RD3: now also U2.9 (A7); no longer U2.11 (B7)
- net RD4: now also U2.7 (A5); no longer U2.13 (B5)
- net RD5: now also U2.2 (A0); no longer U2.18 (B0)
- net RD6: now also U2.4 (A2); no longer U2.16 (B2)
- net RD7: now also U2.6 (A4); no longer U2.14 (B4)
- net ~{INH}: now also U14.4 (Y)

Commit message: more
Connections:
- net RD0: now also U2.9 (A7); no longer U2.5 (A3)
- net RD1: now also U2.8 (A6); no longer U2.3 (A1)
- net RD2: now also U2.7 (A5); no longer U2.8 (A6)
- net RD3: now also U2.6 (A4); no longer U2.9 (A7)
- net RD4: now also U2.5 (A3); no longer U2.7 (A5)
- net RD5: now also U2.4 (A2); no longer U2.2 (A0)
- net RD6: now also U2.3 (A1); no longer U2.4 (A2)
- net RD7: now also U2.2 (A0); no longer U2.6 (A4)
