File: Bus.kicad_sch (KiCad schematic)
At the start: 1 part, among them J1 AppleIIBus

Commit message: schematic and placement done?
Parts:
- added C1, C2, C3, C4: 10u, stdpads:C_0805, symbol Device:C_Small
Connections:
- net +12V: now also C3.1
- net +5V: now also C1.1
- net -12V: now also C2.1
- net -5V: now also C4.1
- net GND: now also C1.2, C2.2, C3.2, C4.2

Commit message: more
Connections:
- net +12V: now also C4.1; no longer C3.1
- net -5V: now also C3.1; no longer C4.1
