File: LEDs.kicad_sch (KiCad schematic)
At the start: 14 parts, among them U26 74AHCT08PW, U27 74AHCT08PW

Commit message: schematic and placement done?
Parts:
- removed R1, R11: 470, stdpads:R_0805, symbol Device:R_Small
- removed U26, U27: 74AHCT08PW, stdpads:TSSOP-14_4.4x5mm_P0.65mm, symbol 74xx:74LS08
- added C20, C21: 2u2, stdpads:C_0603, symbol Device:C_Small
- added R16, R17: 470, stdpads:R_0805, symbol Device:R_Small
- added U7, U8: 74AHCT08PW, stdpads:TSSOP-14_4.4x5mm_P0.65mm, symbol 74xx:74LS08
Connections:
- net +5V: now also C20.1, C21.1, U7.14 (VCC), U8.14 (VCC)
- net ENRD: now also U8.12
- net ENWR: now also U7.9
- net GND: now also C20.2, C21.2, U7.7 (GND), U8.7 (GND)
- net LEDEN: now also U7.10, U7.13, U8.10, U8.13, U8.2, U8.5
- net LED_ACT: now also R17.1; no longer R15.1
- net LED_ENRD: now also R15.1; no longer R13.1
- net LED_ENWR: now also R16.1; no longer R14.1
- net LED_RA14: now also R14.1; no longer R12.1
- net LED_RA15: now also R13.1
- net LED_RA16: now also R12.1
- net RA14: now also U8.9
- net RA15: now also U8.4
- net RA16: now also U8.1
- net RCS: now also U7.12
- net at R12.2: now also U8.3
- net at R13.2: now also U8.6
- net at R15.2: now also U8.11
- net at R14.2: now also U8.8
- new net: R16.2, U7.8
- new net: R17.2, U7.11

Commit message: more
Changed lines of the file:
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@@
 (kicad_sch
-	(version 20231120)
+	(version 20250114)
 	(generator "eeschema")
-	(generator_version "8.0")
+	(generator_version "9.0")
 	(paper "A4")
 	(title_block
@@
 	(label "LED_RA14"
 		(at 146.05 91.44 0)
-		(fields_autoplaced yes)
 		(effects
 			(font
@@
 	(label "LED_RA15"
 		(at 146.05 76.2 0)
-		(fields_autoplaced yes)
 		(effects
 			(font
@@
 	(label "LED_RA16"
 		(at 146.05 60.96 0)
-		(fields_autoplaced yes)
 		(effects
 			(font
@@
 	(label "LED_ENRD"
 		(at 146.05 106.68 0)
-		(fields_autoplaced yes)
 		(effects
 			(font
@@
 	(label "LED_ENWR"
 		(at 146.05 121.92 0)
-		(fields_autoplaced yes)
 		(effects
 			(font
@@
 	(label "LED_ACT"
 		(at 146.05 137.16 0)
-		(fields_autoplaced yes)
 		(effects
 			(font
@@
 		(shape input)
 		(at 125.73 58.42 180)
-		(fields_autoplaced yes)
 		(effects
 			(font
@@
 		(shape input)
 		(at 125.73 78.74 180)
-		(fields_autoplaced yes)
 		(effects
 			(font
@@
 		(shape input)
 		(at 125.73 93.98 180)
-		(fields_autoplaced yes)
 		(effects
 			(font
@@
 		(shape input)
 		(at 125.73 134.62 180)
-		(fields_autoplaced yes)
 		(effects
 			(font
@@
 		(shape input)
 		(at 125.73 124.46 180)
-		(fields_autoplaced yes)
 		(effects
 			(font
@@
 		(shape input)
 		(at 125.73 63.5 180)
-		(fields_autoplaced yes)
 		(effects
 			(font
@@
 		(shape input)
 		(at 125.73 139.7 180)
-		(fields_autoplaced yes)
 		(effects
 			(font
@@
 		(shape input)
 		(at 125.73 109.22 180)
-		(fields_autoplaced yes)
 		(effects
 			(font
@@
 		(shape input)
 		(at 125.73 88.9 180)
-		(fields_autoplaced yes)
 		(effects
 			(font
@@
 		(shape input)
 		(at 125.73 119.38 180)
-		(fields_autoplaced yes)
 		(effects
 			(font
@@
 		(shape input)
 		(at 125.73 104.14 180)
-		(fields_autoplaced yes)
 		(effects
 			(font
@@
 		(shape input)
 		(at 125.73 73.66 180)
-		(fields_autoplaced yes)
-		(effects
-			(font
+		(effects
+			(font
