File: RAM.kicad_sch (KiCad schematic)
At the start: 1 part, among them U1 621024

Commit message: schematic and placement done?
Parts:
- added C5: 10u, stdpads:C_0805, symbol Device:C_Small
Connections:
- net R~{CS} is gone; now on net GND: U1.22 (~{CS})
- net +5V: now also C5.1; no longer U1.30 (CS)
- net A0: now also U1.25 (A11); no longer U1.12 (A0)
- net A1: now also U1.8 (A4); no longer U1.23 (A10)
- net A10: now also U1.31 (A15); no longer U1.28 (A13)
- net A11: now also U1.3 (A14); no longer U1.6 (A6)
- net A13: now also U1.2 (A16); no longer U1.31 (A15)
- net A2: now also U1.26 (A9); no longer U1.11 (A1)
- net A3: now also U1.7 (A5); no longer U1.10 (A2)
- net A4: now also U1.27 (A8); no longer U1.25 (A11)
- net A5: now also U1.6 (A6); no longer U1.9 (A3)
- net A6: now also U1.28 (A13); no longer U1.26 (A9)
- net A7: now also U1.5 (A7); no longer U1.8 (A4)
- net A8: now also U1.23 (A10); no longer U1.27 (A8)
- net A9: now also U1.4 (A12); no longer U1.7 (A5)
- net GND: now also C5.2
- net RA12: now also U1.12 (A0); no longer U1.5 (A7)
- net RA14: now also U1.11 (A1); no longer U1.4 (A12)
- net RA15: now also U1.10 (A2); no longer U1.3 (A14)
- net RA16: now also U1.9 (A3); no longer U1.2 (A16)
- new net RCS: U1.30 (CS)

Commit message: more
Connections:
- net A0: now also U1.23 (A10); no longer U1.25 (A11)
- net A10: now also U1.3 (A14); no longer U1.31 (A15)
- net A11: now also U1.2 (A16); no longer U1.3 (A14)
- net A13: now also U1.31 (A15); no longer U1.2 (A16)
- net A2: now also U1.7 (A5); no longer U1.26 (A9)
- net A3: now also U1.25 (A11); no longer U1.7 (A5)
- net A4: now also U1.6 (A6); no longer U1.27 (A8)
- net A5: now also U1.26 (A9); no longer U1.6 (A6)
- net A6: now also U1.5 (A7); no longer U1.28 (A13)
- net A7: now also U1.27 (A8); no longer U1.5 (A7)
- net A8: now also U1.4 (A12); no longer U1.23 (A10)
- net A9: now also U1.28 (A13); no longer U1.4 (A12)
- net RD0: now also U1.17 (D3); no longer U1.13 (D0)
- net RD1: now also U1.15 (D2); no longer U1.14 (D1)
- net RD2: now also U1.18 (D4); no longer U1.15 (D2)
- net RD3: now also U1.14 (D1); no longer U1.17 (D3)
- net RD4: now also U1.19 (D5); no longer U1.18 (D4)
- net RD5: now also U1.13 (D0); no longer U1.19 (D5)
Changed lines of the file:
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@@
 (kicad_sch
-	(version 20231120)
+	(version 20250114)
 	(generator "eeschema")
-	(generator_version "8.0")
+	(generator_version "9.0")
 	(paper "A4")
 	(title_block
@@
 	)
 	(label "A7"
-		(at 123.19 66.04 0)
-		(fields_autoplaced yes)
+		(at 123.19 68.58 0)
 		(effects
 			(font
@@
 	)
 	(label "RD2"
-		(at 102.87 58.42 180)
-		(fields_autoplaced yes)
+		(at 102.87 63.5 180)
 		(effects
 			(font
@@
 	(label "RD7"
 		(at 102.87 71.12 180)
-		(fields_autoplaced yes)
 		(effects
 			(font
@@
 	)
 	(label "A11"
+		(at 123.19 88.9 0)
+		(effects
+			(font
+				(size 1.27 1.27)
+			)
+			(justify left bottom)
+		)
+	)
+	(label "A6"
+		(at 123.19 66.04 0)
+		(effects
+			(font
+				(size 1.27 1.27)
+			)
+			(justify left bottom)
+		)
+	)
+	(label "RD5"
+		(at 102.87 53.34 180)
+		(effects
+			(font
+				(size 1.27 1.27)
+			)
+			(justify right bottom)
+		)
+	)
+	(label "A10"
 		(at 123.19 83.82 0)
-		(fields_autoplaced yes)
-		(effects
-			(font
-				(size 1.27 1.27)
-			)
-			(justify left bottom)
-		)
-	)
-	(label "A6"
-		(at 123.19 81.28 0)
-		(fields_autoplaced yes)
-		(effects
-			(font
-				(size 1.27 1.27)
-			)
-			(justify left bottom)
-		)
-	)
-	(label "RD5"
-		(at 102.87 66.04 180)
-		(fields_autoplaced yes)
+		(effects
+			(font
+				(size 1.27 1.27)
+			)
+			(justify left bottom)
+		)
+	)
+	(label "A8"
+		(at 123.19 78.74 0)
+		(effects
+			(font
+				(size 1.27 1.27)
+			)
+			(justify left bottom)
+		)
+	)
+	(label "A4"
+		(at 123.19 63.5 0)
+		(effects
+			(font
+				(size 1.27 1.27)
+			)
+			(justify left bottom)
+		)
+	)
+	(label "A2"
+		(at 123.19 60.96 0)
+		(effects
+			(font
+				(size 1.27 1.27)
+			)
+			(justify left bottom)
+		)
+	)
+	(label "A3"
+		(at 123.19 76.2 0)
+		(effects
+			(font
+				(size 1.27 1.27)
+			)
+			(justify left bottom)
+		)
+	)
+	(label "RD0"
+		(at 102.87 60.96 180)
 		(effects
 			(font
@@
 		)
 	)
-	(label "A10"
+	(label "A0"
+		(at 123.19 73.66 0)
+		(effects
+			(font
+				(size 1.27 1.27)
+			)
+			(justify left bottom)
+		)
+	)
+	(label "RD1"
+		(at 102.87 58.42 180)
+		(effects
+			(font
+				(size 1.27 1.27)
+			)
+			(justify right bottom)
+		)
+	)
+	(label "A13"
 		(at 123.19 86.36 0)
-		(fields_autoplaced yes)
-		(effects
-			(font
-				(size 1.27 1.27)
-			)
-			(justify left bottom)
-		)
-	)
-	(label "A8"
-		(at 123.19 73.66 0)
-		(fields_autoplaced yes)
-		(effects
-			(font
-				(size 1.27 1.27)
-			)
-			(justify left bottom)
-		)
-	)
-	(label "A4"
-		(at 123.19 68.58 0)
-		(fields_autoplaced yes)
-		(effects
-			(font
-				(size 1.27 1.27)
-			)
-			(justify left bottom)
-		)
-	)
-	(label "A2"
-		(at 123.19 71.12 0)
-		(fields_autoplaced yes)
-		(effects
-			(font
-				(size 1.27 1.27)
-			)
-			(justify left bottom)
-		)
-	)
-	(label "A3"
-		(at 123.19 60.96 0)
-		(fields_autoplaced yes)
-		(effects
-			(font
-				(size 1.27 1.27)
-			)
-			(justify left bottom)
-		)
-	)
-	(label "RD0"
-		(at 102.87 53.34 180)
-		(fields_autoplaced yes)
-		(effects
-			(font
-				(size 1.27 1.27)
-			)
-			(justify right bottom)
-		)
-	)
-	(label "A0"
-		(at 123.19 76.2 0)
-		(fields_autoplaced yes)
-		(effects
-			(font
-				(size 1.27 1.27)
-			)
-			(justify left bottom)
-		)
-	)
-	(label "RD1"
+		(effects
+			(font
+				(size 1.27 1.27)
+			)
+			(justify left bottom)
+		)
+	)
+	(label "RD3"
 		(at 102.87 55.88 180)
-		(fields_autoplaced yes)
-		(effects
-			(font
-				(size 1.27 1.27)
-			)
-			(justify right bottom)
-		)
-	)
-	(label "A13"
-		(at 123.19 88.9 0)
-		(fields_autoplaced yes)
-		(effects
-			(font
-				(size 1.27 1.27)
-			)
-			(justify left bottom)
-		)
-	)
-	(label "RD3"
-		(at 102.87 60.96 180)
-		(fields_autoplaced yes)
 		(effects
 			(font
@@
 	(label "RD6"
 		(at 102.87 68.58 180)
-		(fields_autoplaced yes)
 		(effects
 			(font
@@
 	)
 	(label "A5"
-		(at 123.19 63.5 0)
-		(fields_autoplaced yes)
+		(at 123.19 71.12 0)
 		(effects
 			(font
@@
 	)
 	(label "RD4"
-		(at 102.87 63.5 180)
-		(fields_autoplaced yes)
+		(at 102.87 66.04 180)
 		(effects
 			(font
@@
 	)
 	(label "A9"
-		(at 123.19 78.74 0)
-		(fields_autoplaced yes)
+		(at 123.19 81.28 0)
 		(effects
 			(font
@@
 	(label "A1"
 		(at 123.19 58.42 0)
-		(fields_autoplaced yes)
 		(effects
 			(font
@@
 		(shape input)
 		(at 123.19 48.26 0)
-		(fields_autoplaced yes)
 		(effects
 			(font
@@
 		(shape input)
 		(at 102.87 78.74 180)
-		(fields_autoplaced yes)
 		(effects
 			(font
@@
 		(shape input)
 		(at 123.19 50.8 0)
-		(fields_autoplaced yes)
 		(effects
 			(font
@@
 		(shape input)
 		(at 102.87 83.82 180)
-		(fields_autoplaced yes)
 		(effects
 			(font
@@
 		(shape input)
 		(at 102.87 81.28 180)
-		(fields_autoplaced yes)
 		(effects
 			(font
@@
 		(shape input)
 		(at 123.19 55.88 0)
-		(fields_autoplaced yes)
 		(effects
 			(font
@@
 		(shape input)
 		(at 134.62 55.88 0)
-		(fields_autoplaced yes)
 		(effects
 			(font
@@
 		(shape bidirectional)
 		(at 93.98 50.8 180)
-		(fields_autoplaced yes)
 		(effects
 			(font
@@
 		(shape input)
 		(at 123.19 53.34 0)
-		(fields_autoplaced yes)
-		(effects
-			(font
+		(effects
+			(font
