File: Registers.kicad_sch (KiCad schematic)
At the start: 4 parts, among them U18 74HCT273PW, U3 74HCT273PW, U4 74HCT273PW, U5 74HCT273PW

Commit message: schematic and placement done?
Parts:
- removed U3, U4: 74HCT273PW, stdpads:TSSOP-20_4.4x6.5mm_P0.65mm, symbol 74xx:74LS273
- added C18, C19: 2u2, stdpads:C_0603, symbol Device:C_Small
- U18, U5: footprint (none) -> stdpads:TSSOP-20_4.4x6.5mm_P0.65mm
Connections:
- net +5V: now also U18.20 (VCC), U5.20 (VCC), C18.1, C19.1
- net A0: now also U18.7 (D2), U5.7 (D2)
- net A1: now also U5.4 (D1)
- net A2clk: now also U5.11 (Cp)
- net A3: now also U18.3 (D0), U5.3 (D0)
- net BankAB: now also U18.2 (Q0)
- net ENRD: now also U18.5 (Q1)
- net ENWR: now also U18.9 (Q3)
- net ENWR1: now also U18.6 (Q2)
- net ENWR1A0: now also U18.8 (D3)
- net GND: now also U18.10 (GND), U18.13 (D4), U18.14 (D5), U18.17 (D6), U18.18 (D7), U5.10 (GND), U5.13 (D4), U5.14 (D5), U5.17 (D6), U5.18 (D7), U5.8 (D3), C18.2, C19.2
- net RA14: now also U5.6 (Q2)
- net RA15: now also U5.5 (Q1)
- net RA16: now also U5.2 (Q0)
- net ~{A0XOR1}: now also U18.4 (D1)
- net ~{A2}clk: now also U18.11 (Cp)
- net ~{RRST}: now also U18.1 (~{Mr}), U5.1 (~{Mr})
Other:
- moved on the sheet: U18
