File: Control.kicad_sch (KiCad schematic)
At the start: 0 parts

Commit message: schematic and placement done?
Parts:
- added C10, C11, C12, C13, C14, C15, C16, C17, C6, C9: 2u2, stdpads:C_0603, symbol Device:C_Small
- added Q1: MMBT3904, stdpads:SOT-23, symbol Transistor_BJT:MMBT3904
- added R1, R3: 10k, stdpads:R_0603, symbol Device:R_Small
- added R2: 2k2, stdpads:R_0603, symbol Device:R_Small
- added R4: 47, stdpads:R_0603, symbol Device:R_Small
- added U10, U15, U4: 74AHC1G14GW, stdpads:SOT-353, symbol GW_Logic:741G04GW
- added U11, U7, U9: 74AHCT08PW, stdpads:TSSOP-14_4.4x5mm_P0.65mm, symbol 74xx:74LS08
- added U12, U13: 74AHCT32PW, stdpads:TSSOP-14_4.4x5mm_P0.65mm, symbol 74xx:74LS32
- added U3: 74AHCT00PW, stdpads:TSSOP-14_4.4x5mm_P0.65mm, symbol 74xx:74LS00
- added U6: 74AHCT02PW, stdpads:TSSOP-14_4.4x5mm_P0.65mm, symbol 74xx:74LS02
Connections:
- new net: U11.8, U13.1
- new net: Q1.1 (B), R2.2, R3.1
- new net: U3.5, U7.6, U9.10
- new net: U13.3, U3.4, U9.9
- new net: Q1.3 (C), R4.2
- new net: U12.9, U6.1
- new net: U11.12, U3.11
- new net: U3.8, U6.11
- new net: U13.2, U7.3
- new net: U11.3, U12.10
- new net: U13.10, U9.3
- new net: U13.9, U6.4
- new net: U7.4, U9.11
- new net: U12.11, U7.5
- new net +5V: C10.1, C11.1, C12.1, C13.1, C14.1, C15.1, C16.1, C17.1, C9.1, R1.1, U10.5 (Vcc), U11.14 (VCC), U12.14 (VCC), U13.14 (VCC), U15.5 (Vcc), U3.14 (VCC), U3.2, U4.5 (Vcc), U6.14 (VCC), U9.14 (VCC)
- new net A0: U6.5, U9.2, U9.5
- new net A1: U6.6, U9.1
- new net A12: U11.1, U12.13
- new net A13: U11.2, U12.12, U6.2
- new net A14: U9.13
- new net A15: U9.12
- new net A2: U3.1
- new net A2clk: U13.6
- new net A2sw: U13.13
- new net BankAB: U6.3
- new net DDIR: U11.6
- new net DMAin: U11.13
- new net DMAinsw: U3.10
- new net DMAout: U11.11
- new net DMAoutEN: U3.13
- new net D~{OE}: U12.3, U12.4
- new net ENRD: U11.10
- new net ENWR: U7.1
- new net ENWR1: U9.4
- new net ENWR1A0: U9.6
- new net GND: C10.2, C11.2, C12.2, C13.2, C14.2, C15.2, C16.2, C17.2, C6.2, C9.2, Q1.2 (E), R3.2, U10.3 (GND), U11.7 (GND), U12.7 (GND), U13.7 (GND), U15.3 (GND), U3.7 (GND), U4.3 (GND), U6.7 (GND), U9.7 (GND)
- new net INH: U3.9, U9.8
- new net INH~{OE}: U3.6
- new net PHI1: U12.2, U6.12
- new net POR: R2.1, U4.4 (Y), U6.8
- new net Q3: U12.1
- new net RA12: U12.8
- new net RCS: U11.5, U3.12, U6.13
- new net RES: U15.4 (Y)
- new net RESsw: U6.9
- new net R~{RST}: U6.10
- new net R~{WE}: U12.6
- new net R~{W}: U10.2 (A), U11.4, U11.9, U12.5
- new net ~{A0XOR1}: U13.8
- new net ~{A2}: U13.4, U3.3
- new net ~{A2}clk: U13.11
- new net ~{DEVSEL}: U13.12, U13.5
- new net ~{POR}: C6.1, R1.2, U4.2 (A)
- new net ~{RESET}: R4.1, U15.2 (A)
- new net ~{R}W: U10.4 (Y), U7.2
- no-connect marks 0 -> 2

Commit message: more
Changed lines of the file:
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@@
 (kicad_sch
-	(version 20231120)
+	(version 20250114)
 	(generator "eeschema")
-	(generator_version "8.0")
+	(generator_version "9.0")
 	(paper "A4")
 	(title_block
@@
 	(label "A1"
 		(at 179.07 74.93 180)
-		(fields_autoplaced yes)
 		(effects
 			(font
@@
 	(label "A12"
 		(at 179.07 24.13 180)
-		(fields_autoplaced yes)
 		(effects
 			(font
@@
 	(label "INH"
 		(at 148.59 119.38 180)
-		(fields_autoplaced yes)
 		(effects
 			(font
@@
 	(label "D~{OE}"
 		(at 102.87 66.04 0)
-		(fields_autoplaced yes)
 		(effects
 			(font
@@
 	(label "A0"
 		(at 179.07 69.85 180)
-		(fields_autoplaced yes)
 		(effects
 			(font
@@
 	(label "~{RESET}"
 		(at 95.25 25.4 180)
-		(fields_autoplaced yes)
 		(effects
 			(font
@@
 	(label "A0"
 		(at 179.07 80.01 180)
-		(fields_autoplaced yes)
 		(effects
 			(font
@@
 	(label "DMAin"
 		(at 194.31 132.08 0)
-		(fields_autoplaced yes)
 		(effects
 			(font
@@
 	(label "A1"
 		(at 179.07 85.09 180)
-		(fields_autoplaced yes)
 		(effects
 			(font
@@
 	(label "DMAoutEN"
 		(at 184.15 129.54 180)
-		(fields_autoplaced yes)
 		(effects
 			(font
@@
 	(label "A0"
 		(at 194.31 92.71 180)
-		(fields_autoplaced yes)
 		(effects
 			(font
@@
 	(label "~{R}W"
 		(at 59.69 119.38 0)
-		(fields_autoplaced yes)
 		(effects
 			(font
@@
 	(label "POR"
 		(at 55.88 30.48 0)
-		(fields_autoplaced yes)
 		(effects
 			(font
@@
 	(label "POR"
 		(at 101.6 40.64 180)
-		(fields_autoplaced yes)
 		(effects
 			(font
@@
 	(label "~{A2}"
 		(at 196.85 44.45 180)
-		(fields_autoplaced yes)
 		(effects
 			(font
@@
 	(label "RCS"
 		(at 184.15 109.22 180)
-		(fields_autoplaced yes)
 		(effects
 			(font
@@
 	(label "~{R}W"
 		(at 95.25 124.46 180)
-		(fields_autoplaced yes)
 		(effects
 			(font
@@
 	(label "A2"
 		(at 179.07 41.91 180)
-		(fields_autoplaced yes)
 		(effects
 			(font
@@
 	(label "A13"
 		(at 179.07 8.89 180)
-		(fields_autoplaced yes)
 		(effects
 			(font
@@
 	(label "PHI1"
 		(at 163.83 127 180)
-		(fields_autoplaced yes)
 		(effects
 			(font
@@
 	(label "A13"
 		(at 95.25 139.7 180)
-		(fields_autoplaced yes)
 		(effects
 			(font
@@
 	(label "A13"
 		(at 179.07 19.05 180)
-		(fields_autoplaced yes)
 		(effects
 			(font
@@
 	(label "A15"
 		(at 95.25 129.54 180)
-		(fields_autoplaced yes)
 		(effects
 			(font
@@
 	(label "~{POR}"
 		(at 35.56 27.94 180)
-		(fields_autoplaced yes)
 		(effects
 			(font
@@
 	(label "A14"
 		(at 95.25 134.62 180)
-		(fields_autoplaced yes)
 		(effects
 			(font
@@
 	(label "R~{W}"
 		(at 184.15 104.14 180)
-		(fields_autoplaced yes)
 		(effects
 			(font
@@
 	(label "RCS"
 		(at 184.15 119.38 180)
-		(fields_autoplaced yes)
 		(effects
 			(font
@@
 	(label "A12"
 		(at 95.25 144.78 180)
-		(fields_autoplaced yes)
 		(effects
 			(font
@@
 	(label "RCS"
 		(at 184.15 124.46 180)
-		(fields_autoplaced yes)
 		(effects
 			(font
@@
 	(label "R~{W}"
 		(at 95.25 109.22 180)
-		(fields_autoplaced yes)
 		(effects
 			(font
@@
 		(shape output)
 		(at 212.09 46.99 0)
-		(fields_autoplaced yes)
 		(effects
 			(font
@@
 		(shape output)
 		(at 212.09 80.01 0)
-		(fields_autoplaced yes)
 		(effects
 			(font
@@
 		(shape input)
 		(at 166.37 13.97 180)
-		(fields_autoplaced yes)
 		(effects
 			(font
@@
 		(shape input)
 		(at 87.63 60.96 180)
-		(fields_autoplaced yes)
 		(effects
 			(font
@@
 		(shape input)
 		(at 166.37 6.35 180)
-		(fields_autoplaced yes)
 		(effects
 			(font
@@
 		(shape output)
 		(at 214.63 129.54 0)
-		(fields_autoplaced yes)
 		(effects
 			(font
@@
 		(shape input)
 		(at 87.63 63.5 180)
-		(fields_autoplaced yes)
 		(effects
 			(font
@@
 		(shape output)
 		(at 64.77 119.38 0)
-		(fields_autoplaced yes)
 		(effects
 			(font
@@
 		(shape input)
 		(at 85.09 119.38 180)
-		(fields_autoplaced yes)
 		(effects
 			(font
@@
 		(shape input)
 		(at 85.09 152.4 180)
-		(fields_autoplaced yes)
 		(effects
 			(font
@@
 		(shape input)
 		(at 166.37 87.63 180)
-		(fields_autoplaced yes)
 		(effects
 			(font
@@
 		(shape input)
 		(at 39.37 116.84 180)
-		(fields_autoplaced yes)
 		(effects
 			(font
@@
 		(shape input)
 		(at 166.37 39.37 180)
-		(fields_autoplaced yes)
 		(effects
 			(font
@@
 		(shape input)
 		(at 85.09 147.32 180)
-		(fields_autoplaced yes)
 		(effects
 			(font
@@
 		(shape input)
 		(at 87.63 68.58 180)
-		(fields_autoplaced yes)
 		(effects
 			(font
@@
 		(shape output)
 		(at 214.63 119.38 0)
-		(fields_autoplaced yes)
 		(effects
 			(font
@@
 		(shape output)
 		(at 116.84 43.18 0)
-		(fields_autoplaced yes)
 		(effects
 			(font
@@
 		(shape output)
 		(at 116.84 27.94 0)
-		(fields_autoplaced yes)
 		(effects
 			(font
@@
 		(shape output)
 		(at 123.19 63.5 0)
-		(fields_autoplaced yes)
 		(effects
 			(font
@@
 		(shape output)
 		(at 214.63 134.62 0)
-		(fields_autoplaced yes)
 		(effects
 			(font
@@
 		(shape output)
 		(at 212.09 57.15 0)
-		(fields_autoplaced yes)
 		(effects
 			(font
@@
 		(shape output)
 		(at 123.19 71.12 0)
-		(fields_autoplaced yes)
 		(effects
 			(font
@@
 		(shape output)
 		(at 209.55 16.51 0)
-		(fields_autoplaced yes)
 		(effects
 			(font
@@
 		(shape input)
 		(at 85.09 127 180)
-		(fields_autoplaced yes)
 		(effects
 			(font
@@
 		(shape input)
 		(at 85.09 104.14 180)
-		(fields_autoplaced yes)
 		(effects
 			(font
@@
 		(shape input)
 		(at 85.09 114.3 180)
-		(fields_autoplaced yes)
 		(effects
 			(font
@@
 		(shape input)
 		(at 101.6 45.72 180)
-		(fields_autoplaced yes)
 		(effects
 			(font
@@
 		(shape output)
 		(at 214.63 106.68 0)
-		(fields_autoplaced yes)
 		(effects
 			(font
@@
 		(shape input)
 		(at 85.09 149.86 180)
-		(fields_autoplaced yes)
 		(effects
 			(font
@@
 		(shape input)
 		(at 166.37 52.07 180)
-		(fields_autoplaced yes)
 		(effects
 			(font
@@
 		(shape input)
 		(at 85.09 154.94 180)
-		(fields_autoplaced yes)
 		(effects
 			(font
@@
 		(shape output)
 		(at 212.09 90.17 0)
-		(fields_autoplaced yes)
 		(effects
 			(font
@@
 		(shape input)
 		(at 166.37 59.69 180)
-		(fields_autoplaced yes)
 		(effects
 			(font
@@
 		(shape tri_state)
 		(at 116.84 15.24 0)
-		(fields_autoplaced yes)
-		(effects
-			(font
+		(effects
+			(font

Commit message: more
Connections:
- net A12: now also U12.9; no longer U12.13
- net A13: now also U12.10; no longer U12.12
- net A14: now also U9.10; no longer U9.13
- net A15: now also U9.9; no longer U9.12
- net INH: now also U9.11; no longer U9.8
- net RA12: now also U12.11; no longer U12.8
- net at U3.5, U7.6: now also U9.12; no longer U9.10
- net at U13.3, U3.4: now also U9.13; no longer U9.9
- net at U6.1: now also U12.13; no longer U12.9
- net at U11.3: now also U12.12; no longer U12.10
- net at U7.4: now also U9.8; no longer U9.11
- net at U7.5: now also U12.8; no longer U12.11
Other:
- moved on the sheet: U12C, U12D, U9C, U9D
Changed lines of the file:
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@@
 	(symbol
 		(lib_id "74xx:74LS08")
-		(at 138.43 119.38 0)
+		(at 102.87 132.08 0)
 		(unit 3)
 		(exclude_from_sim no)
@@
 		(dnp no)
 		(property "Reference" "U9"
-			(at 138.43 119.38 0)
+			(at 102.87 132.08 0)
 			(effects
 				(font
@@
 		)
 		(property "Value" "74AHCT08PW"
-			(at 138.43 114.3 0)
+			(at 102.87 127 0)
 			(effects
 				(font
@@
 		)
 		(property "Footprint" "stdpads:TSSOP-14_4.4x5mm_P0.65mm"
-			(at 138.43 119.38 0)
+			(at 102.87 132.08 0)
 			(effects
 				(font
@@
 		)
 		(property "Datasheet" "http://www.ti.com/lit/gpn/sn74LS08"
-			(at 138.43 119.38 0)
+			(at 102.87 132.08 0)
 			(effects
 				(font
@@
 		)
 		(property "Description" ""
-			(at 138.43 119.38 0)
+			(at 102.87 132.08 0)
 			(effects
 				(font
@@
 		)
 		(property "LCSC Part" "C155175"
-			(at 138.43 119.38 0)
+			(at 102.87 132.08 0)
 			(effects
 				(font
@@
 	(symbol
 		(lib_id "74xx:74LS32")
-		(at 201.93 16.51 0)
+		(at 102.87 142.24 0)
+		(mirror x)
 		(unit 3)
 		(exclude_from_sim no)
@@
 		(dnp no)
 		(property "Reference" "U12"
-			(at 201.93 16.51 0)
+			(at 102.87 142.24 0)
 			(effects
 				(font
@@
 		)
 		(property "Value" "74AHCT32PW"
-			(at 201.93 11.43 0)
+			(at 102.87 137.16 0)
 			(effects
 				(font
@@
 		)
 		(property "Footprint" "stdpads:TSSOP-14_4.4x5mm_P0.65mm"
-			(at 201.93 16.51 0)
+			(at 102.87 142.24 0)
 			(effects
 				(font
@@
 		)
 		(property "Datasheet" "http://www.ti.com/lit/gpn/sn74LS32"
-			(at 201.93 16.51 0)
+			(at 102.87 142.24 0)
 			(effects
 				(font
@@
 		)
 		(property "Description" ""
-			(at 201.93 16.51 0)
+			(at 102.87 142.24 0)
 			(effects
 				(font
@@
 		)
 		(property "LCSC Part" "C129435"
-			(at 201.93 16.51 0)
+			(at 102.87 142.24 0)
 			(effects
 				(font
@@
 	(symbol
 		(lib_id "74xx:74LS32")
-		(at 102.87 142.24 0)
+		(at 201.93 16.51 0)
+		(mirror x)
 		(unit 4)
 		(exclude_from_sim no)
@@
 		(dnp no)
 		(property "Reference" "U12"
-			(at 102.87 142.24 0)
+			(at 201.93 16.51 0)
 			(effects
 				(font
@@
 		)
 		(property "Value" "74AHCT32PW"
-			(at 102.87 137.16 0)
+			(at 201.93 11.43 0)
 			(effects
 				(font
@@
 		)
 		(property "Footprint" "stdpads:TSSOP-14_4.4x5mm_P0.65mm"
-			(at 102.87 142.24 0)
+			(at 201.93 16.51 0)
 			(effects
 				(font
@@
 		)
 		(property "Datasheet" "http://www.ti.com/lit/gpn/sn74LS32"
-			(at 102.87 142.24 0)
+			(at 201.93 16.51 0)
 			(effects
 				(font
@@
 		)
 		(property "Description" ""
-			(at 102.87 142.24 0)
+			(at 201.93 16.51 0)
 			(effects
 				(font
@@
 		)
 		(property "LCSC Part" "C129435"
-			(at 102.87 142.24 0)
+			(at 201.93 16.51 0)
 			(effects
 				(font
@@
 	(symbol
 		(lib_id "74xx:74LS08")
-		(at 102.87 132.08 0)
+		(at 138.43 119.38 0)
+		(mirror x)
 		(unit 4)
 		(exclude_from_sim no)
@@
 		(dnp no)
 		(property "Reference" "U9"
-			(at 102.87 132.08 0)
+			(at 138.43 119.38 0)
 			(effects
 				(font
@@
 		)
 		(property "Value" "74AHCT08PW"
-			(at 102.87 127 0)
+			(at 138.43 114.3 0)
 			(effects
 				(font
@@
 		)
 		(property "Footprint" "stdpads:TSSOP-14_4.4x5mm_P0.65mm"
-			(at 102.87 132.08 0)
+			(at 138.43 119.38 0)
 			(effects
 				(font
@@
 		)
 		(property "Datasheet" "http://www.ti.com/lit/gpn/sn74LS08"
-			(at 102.87 132.08 0)
+			(at 138.43 119.38 0)
 			(effects
 				(font
@@
 		)
 		(property "Description" ""
-			(at 102.87 132.08 0)
+			(at 138.43 119.38 0)
 			(effects
 				(font
@@
 		)
 		(property "LCSC Part" "C155175"
-			(at 102.87 132.08 0)
+			(at 138.43 119.38 0)
 			(effects
 				(font
